File: DisplayDriver/DisplayDriver.kicad_pcb (KiCad board)
At the start: 2 copper layers, 50 parts, among them J1 HTSS-108-01-G-D, J3 SAMTEC_HTSS-108-01-G-D, SW1 Generic (Lab Kit), U1 ESP32-S3-WROOM-1, U2 74AHCT245, U3 74AHCT245, U4 AP2112K-3.3TRG1, U5 STUSB4500QTR, X1 CUI_UJ20-C-H-G-SMT-TR, X2 CUI_UJ20-C-H-G-SMT-TR

Commit message: PCB wiring
Parts:
- removed C11, C12: 10uF, Capacitor_SMD:C_0805_2012Metric_Pad1.18x1.45mm_HandSolder
- added C17: 0.1uF, Capacitor_SMD:C_0603_1608Metric, F.Cu at (101.7, 85.8)
- added J2: HEADER-1X14, Connector_PinHeader_2.54mm:PinHeader_1x14_P2.54mm_Vertical, F.Cu at (105.0, 122.8)
- added PC2: 1000uF/6.3V, Capacitor_SMD:C_0805_2012Metric_Pad1.18x1.45mm_HandSolder, F.Cu at (177.2, 78.3)
- added R10: 33, Resistor_SMD:R_0805_2012Metric_Pad1.20x1.40mm_HandSolder, F.Cu at (88.2, 84.0)
- added R11: 33, Resistor_SMD:R_0805_2012Metric_Pad1.20x1.40mm_HandSolder, F.Cu at (98.5, 96.8)
- added R12: 22, Resistor_SMD:R_0603_1608Metric, F.Cu at (125.7, 93.8)
- added R13: 22, Resistor_SMD:R_0603_1608Metric, F.Cu at (125.7, 98.2)
- added R14: 22, Resistor_SMD:R_0603_1608Metric, F.Cu at (124.2, 102.8)
- added R15: 22, Resistor_SMD:R_0603_1608Metric, F.Cu at (124.2, 106.5)
- added R16: 22, Resistor_SMD:R_0603_1608Metric, F.Cu at (121.1, 111.8)
- added R17: 22, Resistor_SMD:R_0603_1608Metric, F.Cu at (121.0, 115.0)
- added R18: 22, Resistor_SMD:R_0603_1608Metric, F.Cu at (146.2, 75.8)
- added R19: 22, Resistor_SMD:R_0603_1608Metric, F.Cu at (146.2, 79.8)
- added R20: 22, Resistor_SMD:R_0603_1608Metric, F.Cu at (146.5, 83.8)
- added R21: 22, Resistor_SMD:R_0603_1608Metric, F.Cu at (146.5, 89.0)
- added R22: 22, Resistor_SMD:R_0603_1608Metric, F.Cu at (145.8, 94.1)
- C1, C15, C16, C5: footprint Capacitor_SMD:C_0805_2012Metric_Pad1.18x1.45mm_HandSolder -> Capacitor_SMD:C_0603_1608Metric
- C10, C9: value 0.1uF -> 100uF
- C13: value 10uF -> 100uF
- C2: value 10uF -> 0.1uF; footprint Capacitor_SMD:C_0805_2012Metric_Pad1.18x1.45mm_HandSolder -> Capacitor_SMD:C_0603_1608Metric
- DOWN1, RST1, UP1: value SW_TL3330AF260QG -> TL3330AF260QG
- LED1: value LED_WS2812B_PLCC4_5.0x5.0mm_P3.2mm -> WS2812B_3535FULL
- R3: value 10K -> 33; footprint Resistor_SMD:R_0805_2012Metric_Pad1.20x1.40mm_HandSolder -> Resistor_SMD:R_0603_1608Metric
- R7: value Resistor_SMD:R_0805_2012Metric_Pad1.20x1.40mm_HandSolder -> 330
- SW1: value Generic (Lab Kit) -> (Generic) Lab Kit
- moved R2 147.6 mm to (78.5, 107.2), turned to -90 degrees
- moved C15 142.0 mm to (78.2, 121.0), turned to -90 degrees
- moved R24 139.2 mm to (94.0, 113.0), turned to 90 degrees
- moved R8 136.4 mm to (88.5, 93.2), turned to -90 degrees
- moved PC1 132.7 mm to (83.0, 113.5), turned to 90 degrees
- moved R3 132.4 mm to (88.8, 77.2), turned to -90 degrees
- moved C3 130.3 mm to (78.5, 113.5), turned to 90 degrees
- moved R23 128.9 mm to (94.0, 119.5), turned to -90 degrees
- moved R27 128.3 mm to (93.0, 96.2), turned to 90 degrees
- moved C6 121.0 mm to (83.2, 107.2), turned to -90 degrees
- moved R6 114.6 mm to (107.0, 98.5), turned to 90 degrees
- moved C5 110.5 mm to (98.2, 119.7), turned to -90 degrees
- moved C4 109.9 mm to (98.5, 113.8), turned to 90 degrees
- moved R7 105.9 mm to (115.2, 94.5)
- moved C14 105.3 mm to (111.5, 99.7), turned to 90 degrees
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- renumbered L1 to D1, L2 to D2, L3 to D3, R8 to R23, R8 to R24, R8 to R25, R8 to R26, R9 to R27, R9 to R28, R9 to R29, R9 to R8
Connections:
- C1 pad 1: GND -> +5V
- C1 pad 2: +5V -> GND
- C10 pad 2: 3.3V -> +5V
- C13 pad 1: 3.3V -> GND
- C13 pad 2: GND -> 3.3V
- C14 pad 1: 3.3V -> GND
- C14 pad 2: GND -> +5V
- C15 pad 1: GND -> +5V
- C15 pad 2: 3.3V -> GND
- C2 pad 1: GND -> +5V
- C2 pad 2: +5V -> GND
- C5 pad 1: GND -> 3.3V
- C5 pad 2: 3.3V -> GND
- C7 pad 1: 3.3V -> GND
- C7 pad 2: GND -> 3.3V
- C8 pad 1: 3.3V -> GND
- C8 pad 2: GND -> 3.3V
- C9 pad 2: 3.3V -> +5V
- D1 pad 1: (no net) -> Net-(D1-K)
- D1 pad 2: (no net) -> /D13
- D2 pad 1: (no net) -> GND
- D2 pad 2: (no net) -> Net-(D2-A)
- D3 pad 1: (no net) -> Net-(D3-K)
- D3 pad 2: (no net) -> 3.3V
- DOWN1 pad 1: (no net) -> GND
- DOWN1 pad 2: (no net) -> /DOWN
- DOWN1 pad S1: (no net) -> unconnected-(DOWN1-PadS1)
- DOWN1 pad S2: (no net) -> unconnected-(DOWN1-PadS2)
- LED1 pad 1: (no net) -> Net-(LED1-DI)
- LED1 pad 2: (no net) -> 3.3V
- LED1 pad 3: (no net) -> unconnected-(LED1-DO-Pad3)
- LED1 pad 4: (no net) -> GND
- R23 pad 1: GND -> /CC2A
- R25 pad 1: GND -> /CC2B
- R26 pad 1: GND -> /CC1B
- R27 pad 1: Net-(X1-DN1) -> /DP_A
- R27 pad 2: Net-(R9B-1) -> /DA+
- R28 pad 1: Net-(X1-DN1) -> /DN_B
- R28 pad 2: Net-(R9B-1) -> /DB-
- R29 pad 1: Net-(X1-DN1) -> /DP_B
- R29 pad 2: Net-(R9B-1) -> /DB+
- R3 pad 1: 3.3V -> /CLK_3V
- R3 pad 2: unconnected-(R3-Pad2) -> Net-(U3-A3)
- R4 pad 2: Net-(L2-PadA) -> Net-(D2-A)
- R5 pad 1: Net-(L3-PadC) -> Net-(D3-K)
- R6 pad 1: Net-(L1-PadC) -> Net-(D1-K)
- R8 pad 1: Net-(X1-DN1) -> /DN_A
- R8 pad 2: Net-(R9B-1) -> /DA-
- RST1 pad 1: (no net) -> GND
- RST1 pad 2: (no net) -> /~{RESET}
- SJ1 pad 1: (no net) -> /M1_E8
- SJ1 pad 2: (no net) -> /M1_E
- SW1 pad 1: (no net) -> /BOOT0
- SW1 pad 2: (no net) -> GND
- U1 pad 13: /D1- -> /DA-
- U1 pad 14: /D1+ -> /DA+
- U2 pad 12: /M1_B2 -> Net-(U2-B7)
- U2 pad 13: /M1_G2 -> Net-(U2-B6)
- U2 pad 14: /M1_R2 -> Net-(U2-B5)
- U2 pad 15: /M1_B1 -> Net-(U2-B4)
- U2 pad 16: /M1_G1 -> Net-(U2-B3)
- U2 pad 17: /M1_R1 -> Net-(U2-B2)
- U2 pad 2: /LAT_3V -> Net-(U2-A1)
- U2 pad 9: /OE_3V -> Net-(U2-A8)
- U3 pad 11: /M1_A -> Net-(U3-B8)
- U3 pad 12: /M1_B -> Net-(U3-B7)
- U3 pad 13: /M1_C -> Net-(U3-B6)
- U3 pad 14: /M1_D -> Net-(U3-B5)
- U3 pad 15: /M1_E -> Net-(U3-B4)
- U3 pad 4: /CLK_3V -> Net-(U3-A3)
- U4 pad 4: (no net) -> unconnected-(U4-NC-Pad4)
- U5 pad 10: Net-(U5-GND-Pad10) -> unconnected-(U5-GND-Pad10)_1
- U5 pad 25: Net-(U5-GND-Pad10) -> unconnected-(U5-GND-Pad10)
- UP1 pad 1: (no net) -> GND
- UP1 pad 2: (no net) -> /UP
- UP1 pad S1: (no net) -> unconnected-(UP1-PadS1)
- UP1 pad S2: (no net) -> unconnected-(UP1-PadS2)
- X1 pad A1: (no net) -> GND
- X1 pad A12: (no net) -> GND
- X1 pad A4: (no net) -> +5V
- X1 pad A5: (no net) -> /CC1A
- X1 pad A6: (no net) -> /DP_A
- X1 pad A7: (no net) -> /DN_A
- X1 pad A9: (no net) -> +5V
- X1 pad B12: (no net) -> GND
- X1 pad B4: (no net) -> +5V
- X1 pad B5: (no net) -> GND
- X1 pad B6: (no net) -> /DP_A
- X1 pad B7: (no net) -> /DN_A
- X1 pad B9: (no net) -> +5V
- X1 pad SH1: (no net) -> GND
- X1 pad SH2: (no net) -> GND
- X1 pad SH3: (no net) -> GND
- X1 pad SH4: (no net) -> GND
- X2 pad A1: (no net) -> GND
- X2 pad A12: (no net) -> GND
- X2 pad A5: (no net) -> /CC1B
- X2 pad A6: (no net) -> /DP_B
- X2 pad A7: (no net) -> /DN_B
- X2 pad B1: (no net) -> GND
- X2 pad B12: (no net) -> GND
- X2 pad B5: (no net) -> /CC2B
- X2 pad B6: (no net) -> /DP_B
- X2 pad B7: (no net) -> /DN_B
- X2 pad SH1: (no net) -> GND
- X2 pad SH2: (no net) -> GND
- X2 pad SH3: (no net) -> GND
- X2 pad SH4: (no net) -> GND
Routing:
- net /BOOT0: track 2.43 -> 98.6 mm, vias 0 -> 2
- net /~{RESET}: track 0.00 -> 84.2 mm
- net (no net): track 86.3 -> 8.82 mm
- net +5V: track 0.00 -> 69.4 mm, vias 0 -> 1
- net /NEOPIX: track 2.61 -> 65.7 mm, vias 0 -> 3
- net /UART_TX: track 8.80 -> 69.2 mm, vias 0 -> 2
- net /UART_RX: track 9.61 -> 66.3 mm, vias 0 -> 2
- net Net-(LED1-DI): track 0.00 -> 47.8 mm, vias 0 -> 2
- net /DOWN: track 8.89 -> 54.7 mm, vias 0 -> 2
- net 3.3V: track 0.00 -> 45.2 mm
- net Net-(U3-A3): track 0.00 -> 44.2 mm, vias 0 -> 2
- net Net-(U2-A8): track 0.00 -> 41.9 mm
- net /OE_3V: track 44.8 -> 4.01 mm
- net /CLK_3V: track 44.1 -> 4.51 mm, vias 2 -> 0
- net /UP: track 8.07 -> 45.4 mm, vias 0 -> 2
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
Commit message: packaging review submission +gerbers
Parts:
- removed C10, C9: 100uF, Capacitor_SMD:C_0805_2012Metric_Pad1.18x1.45mm_HandSolder
- removed J3: SAMTEC_HTSS-108-01-G-D, DisplayDriver:SAMTEC_HTSS-108-01-G-D
- removed PC2: 1000uF/6.3V, Capacitor_SMD:C_0805_2012Metric_Pad1.18x1.45mm_HandSolder
- removed U5: STUSB4500QTR, Package_DFN_QFN:QFN-24-1EP_4x4mm_P0.5mm_EP2.7x2.7mm
- SJ1: value SolderJumper-3_P1.3mm_Open_Rounded -> SOLDERJUMPER_2WAY
- X1, X2: value CUI_UJ20-C-H-G-SMT-TR -> UJ20-C-H-G-SMT-TR
- moved C8 24.3 mm to (83.8, 72.5)
- moved C7 24.2 mm to (83.8, 76.2)
- moved C17 18.6 mm to (83.8, 81.0), turned to 180 degrees
- moved C2 11.8 mm to (116.0, 99.5), turned to -90 degrees
- moved C1 11.1 mm to (124.8, 73.0), turned to -90 degrees
- moved DOWN1 1.75 mm to (77.5, 98.4)
- moved RST1 1.75 mm to (77.5, 78.4)
- moved UP1 1.75 mm to (77.6, 88.4)
- turned R24 to -90 degrees
- turned R26 to -90 degrees
- turned R6 to -90 degrees
Connections:
- RST1 pad S1: (no net) -> unconnected-(RST1-PadS1)
- RST1 pad S2: (no net) -> unconnected-(RST1-PadS2)
- X1 pad A8: (no net) -> unconnected-(X1-SBU1-PadA8)
- X1 pad B5: GND -> /CC2A
- X1 pad B8: (no net) -> unconnected-(X1-SBU2-PadB8)
- X1 pad SH1: GND -> unconnected-(X1-SHIELD-PadSH1)_1
- X1 pad SH2: GND -> unconnected-(X1-SHIELD-PadSH1)_3
- X1 pad SH3: GND -> unconnected-(X1-SHIELD-PadSH1)
- X1 pad SH4: GND -> unconnected-(X1-SHIELD-PadSH1)_2
- X2 pad A4: (no net) -> Net-(X2-VBUS-PadA4)
- X2 pad A8: (no net) -> unconnected-(X2-SBU1-PadA8)
- X2 pad A9: (no net) -> Net-(X2-VBUS-PadA4)
- X2 pad B4: (no net) -> Net-(X2-VBUS-PadA4)
- X2 pad B8: (no net) -> unconnected-(X2-SBU2-PadB8)
- X2 pad B9: (no net) -> Net-(X2-VBUS-PadA4)
Routing:
- net GND: track 36.1 -> 356.6 mm, vias 3 -> 4
- net 3.3V: track 45.2 -> 58.1 mm
- net +5V: track 69.4 -> 79.6 mm
- net Net-(X2-VBUS-PadA4): track 0.00 -> 8.82 mm
- net (no net): track 8.82 -> 0.00 mm
- net /UP: track 45.4 -> 50.2 mm
- net /DOWN: track 54.7 -> 58.3 mm
- net /BOOT0: track 98.6 -> 96.4 mm, vias 2 -> 1
- net Net-(U3-A3): track 44.2 -> 42.1 mm
- net /DP_A: track 26.9 -> 28.8 mm, vias 4 -> 2
- net unconnected-(U1-IO35-Pad28): track 12.9 -> 11.0 mm
- net Net-(D1-K): track 5.73 -> 4.34 mm
- net unconnected-(U1-IO36-Pad29): track 11.7 -> 10.5 mm
- net /DN_A: track 31.3 -> 32.5 mm
- net /CC1A: track 13.2 -> 13.9 mm
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- added copper zone on B.Cu, net GND
