File: DisplayDriver/DisplayDriver.kicad_pcb (KiCad board)
At the start: 2 copper layers, 100 x 75 mm, 39 parts, among them J1 HTSS-108-01-G-D, J2 HEADER-1X14, U1 ESP32-S3-WROOM-1, U2 74AHCT245, U3 74AHCT245, U4 AMS1117-3.3, X2 UJ20-C-H-G-SMT-TR

Commit message: JLCPCB audit correction
Parts:
- moved D1 1.80 mm to (92.2, 89.9)
Routing:
- net Net-(D1-K): track 4.45 -> 6.25 mm
- net /D9: track 46.1 -> 45.3 mm
- net 3.3V: track 182.3 -> 182.9 mm
Other:
- board text added: "AVIATOR v1.0"
Changed lines of the file:
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@@
 		(grid_origin 50.225 99.825)
 		(pcbplotparams
-			(layerselection 0x00010f0_ffffffff)
+			(layerselection 0x00010fc_ffffffff)
 			(plot_on_all_layers_selection 0x0000000_00000000)
 			(disableapertmacros no)
@@
 			(drillshape 0)
 			(scaleselection 1)
-			(outputdirectory "")
+			(outputdirectory "Gerbers/")
 		)
 	)
@@
 		)
 		(property "Value" "HEADER-1X14"
-			(at 2.55 26.175 180)
+			(at -2.65 29.475 180)
 			(layer "F.Fab")
 			(effects
@@
 		)
 		(fp_text user "KEEP-OUT ZONE"
-			(at 0 -18.92 0)
+			(at 7.5 -15.35 0)
 			(layer "Cmts.User")
+			(hide yes)
 			(effects
 				(font
@@
 	(footprint "LED_SMD:LED_0603_1608Metric"
 		(layer "F.Cu")
-		(at 94.025 89.925 -90)
+		(at 92.225 89.925 -90)
 		(descr "LED SMD 0603 (1608 Metric), square (rectangular) end terminal, IPC_7351 nominal, (Body size source: http://www.tortai-tech.com/upload/download/2011102023233369053.pdf), generated with kicad-footprint-generator")
 		(tags "LED")
@@
 		(layer "Edge.Cuts")
 	)
+	(gr_text "AVIATOR v1.0\n"
+		(at 93.725 93.825 0)
+		(layer "F.SilkS")
+		(effects
+			(font
+				(face "Agency FB")
+				(size 3 3)
+				(thickness 0.25)
+				(bold yes)
+			)
+			(justify left bottom)
+		)
+		(render_cache "AVIATOR v1.0\n" 0
+			(polygon
+				(pts
+					(xy 95.553157 93.315) (xy 95.074685 93.315) (xy 94.977965 92.752264) (xy 94.374197 92.752264) (xy 94.277477 93.315)
+					(xy 93.801203 93.315) (xy 93.801203 93.306939) (xy 93.999188 92.283318) (xy 94.437944 92.283318)
+					(xy 94.909822 92.283318) (xy 94.675348 90.827386) (xy 94.437944 92.283318) (xy 93.999188 92.283318)
+					(xy 94.425488 90.07927) (xy 94.932536 90.07927)
+				)
+			)
+			(polygon
+				(pts
+					(xy 97.417219 90.07927) (xy 96.799528 93.315) (xy 96.318859 93.315) (xy 95.702634 90.07927) (xy 96.186967 90.07927)
+					(xy 96.54747 92.294309) (xy 96.554396 92.447151) (xy 96.559926 92.57128) (xy 96.564105 92.418437)
+					(xy 96.572383 92.294309) (xy 96.935083 90.07927)
+				)
+			)
+			(polygon
+				(pts
+					(xy 98.169731 93.315) (xy 97.687595 93.315) (xy 97.687595 90.07927) (xy 98.169731 90.07927)
+				)
+			)
+			(polygon
+				(pts
+					(xy 100.192794 93.315) (xy 99.714323 93.315) (xy 99.617602 92.752264) (xy 99.013834 92.752264)
+					(xy 98.917114 93.315) (xy 98.44084 93.315) (xy 98.44084 93.306939) (xy 98.638825 92.283318) (xy 99.077581 92.283318)
+					(xy 99.549459 92.283318) (xy 99.314986 90.827386) (xy 99.077581 92.283318) (xy 98.638825 92.283318)
+					(xy 99.065125 90.07927) (xy 99.572173 90.07927)
+				)
+			)
+			(polygon
+				(pts
+					(xy 101.853157 90.548217) (xy 101.321196 90.548217) (xy 101.321196 93.315) (xy 100.841259 93.315)
+					(xy 100.841259 90.548217) (xy 100.309298 90.548217) (xy 100.309298 90.07927) (xy 101.853157 90.07927)
+				)
+			)
+			(polygon
+				(pts
+					(xy 103.577568 90.104243) (xy 103.692627 90.211377) (xy 103.715753 90.334993) (xy 103.715753 93.059277)
+					(xy 103.681207 93.204869) (xy 103.56472 93.294771) (xy 103.423394 93.315) (xy 102.376325 93.315)
+					(xy 102.225243 93.290027) (xy 102.112491 93.182893) (xy 102.089829 93.059277) (xy 102.089829 92.846053)
+					(xy 102.572697 92.846053) (xy 103.233618 92.846053) (xy 103.233618 90.548217) (xy 102.572697 90.548217)
+					(xy 102.572697 92.846053) (xy 102.089829 92.846053) (xy 102.089829 90.334993) (xy 102.123682 90.189401)
+					(xy 102.250983 90.095253) (xy 102.376325 90.07927) (xy 103.423394 90.07927)
+				)
+			)
+			(polygon
+				(pts
+					(xy 105.74248 93.315) (xy 105.239829 93.315) (xy 104.707868 91.822431) (xy 104.707868 91.672913)
+					(xy 104.707868 91.533004) (xy 105.181943 91.533004) (xy 105.181943 90.548217) (xy 104.574511 90.548217)
+					(xy 104.574511 93.315) (xy 104.091643 93.315) (xy 104.091643 90.07927) (xy 105.37172 90.07927)
+					(xy 105.52512 90.104243) (xy 105.639603 90.211377) (xy 105.662613 90.334993) (xy 105.662613 91.558649)
+					(xy 105.628175 91.704462) (xy 105.52486 91.78726) (xy 105.378246 91.809897) (xy 105.226021 91.814345)
+					(xy 105.211252 91.814371)
+				)
+			)
+			(polygon
+				(pts
+					(xy 108.275523 91.251636) (xy 107.744295 93.315) (xy 107.292934 93.315) (xy 106.760973 91.251636)
+					(xy 107.245307 91.251636) (xy 107.519347 92.61158) (xy 107.793387 91.251636)
+				)
+			)
+			(polygon
+				(pts
+					(xy 109.106437 93.315) (xy 108.632362 93.315) (xy 108.632362 91.017163) (xy 108.446981 91.017163)
+					(xy 108.446981 90.946821) (xy 108.696842 90.07927) (xy 109.106437 90.07927)
+				)
+			)
+			(polygon
+				(pts
+					(xy 109.935153 93.315) (xy 109.471336 93.315) (xy 109.471336 92.799159) (xy 109.935153 92.799159)
+				)
+			)
+			(polygon
+				(pts
+					(xy 111.72435 90.104243) (xy 111.838544 90.211377) (xy 111.861496 90.334993) (xy 111.861496 93.059277)
+					(xy 111.82721 93.204869) (xy 111.698281 93.299017) (xy 111.571336 93.315) (xy 110.5653 93.315)
+					(xy 110.414217 93.290027) (xy 110.301465 93.182893) (xy 110.278803 93.059277) (xy 110.278803 92.846053)
+					(xy 110.752878 92.846053) (xy 111.389619 92.846053) (xy 111.389619 90.548217) (xy 110.752878 90.548217)
+					(xy 110.752878 92.846053) (xy 110.278803 92.846053) (xy 110.278803 90.334993) (xy 110.313436 90.189401)
+					(xy 110.430214 90.099498) (xy 110.571894 90.07927) (xy 111.571336 90.07927)
+				)
+			)
+		)
+	)
 	(dimension
 		(type aligned)
@@
 	)
 	(segment
-		(start 68.475 49.955)
-		(end 67.495 49.955)
+		(start 67.495 49.955)
+		(end 63.225 54.225)
 		(width 0.2)
 		(layer "F.Cu")
@@
 	)
 	(segment
-		(start 77.825 71.925)
-		(end 80.25 74.35)
+		(start 63.225 54.225)
+		(end 63.225 64.5875)
 		(width 0.2)
 		(layer "F.Cu")
@@
 	)
 	(segment
-		(start 80.25 74.35)
-		(end 80.25 95.675)
+		(start 63.225 64.5875)
+		(end 65.825 67.1875)
 		(width 0.2)
 		(layer "F.Cu")
@@
 	)
 	(segment
-		(start 63.825 53.625)
-		(end 63.825 65.1875)
+		(start 77.825 71.925)
+		(end 80.25 74.35)
 		(width 0.2)
 		(layer "F.Cu")
@@
 	)
 	(segment
-		(start 67.495 49.955)
-		(end 63.825 53.625)
+		(start 80.25 74.35)
+		(end 80.25 95.675)
 		(width 0.2)
 		(layer "F.Cu")
@@
 	)
 	(segment
-		(start 63.825 65.1875)
-		(end 65.825 67.1875)
+		(start 68.475 49.955)
+		(end 67.495 49.955)
 		(width 0.2)
 		(layer "F.Cu")
@@
 	)
 	(segment
+		(start 62.225 53.325)
+		(end 63.025 52.525)
+		(width 0.2)
+		(layer "F.Cu")
+		(net 24)
+	)
+	(segment
 		(start 54.0375 49.075)
 		(end 58.0225 49.075)
@@
 	)
 	(segment
+		(start 62.225 71.4625)
+		(end 62.225 53.325)
+		(width 0.2)
+		(layer "F.Cu")
+		(net 24)
+	)
+	(segment
 		(start 77.325 46.525)
 		(end 101.325 46.525)
@@
 	(segment
 		(start 65.825 75.0625)
-		(end 63.025 72.2625)
+		(end 62.225 71.4625)
 		(width 0.2)
 		(layer "F.Cu")
@@
 	)
 	(segment
-		(start 63.025 72.2625)
-		(end 63.025 52.525)
-		(width 0.2)
-		(layer "F.Cu")
-		(net 24)
-	)
-	(segment
 		(start 94.325 83.775)
 		(end 94.375 83.725)
@@
 	)
 	(segment
-		(start 94.025 89.1375)
-		(end 94.125 89.0375)
+		(start 92.325 89.0375)
+		(end 98.4125 89.0375)
 		(width 0.2)
 		(layer "F.Cu")
@@
 	)
 	(segment
-		(start 94.125 89.0375)
-		(end 98.4125 89.0375)
+		(start 98.4125 89.0375)
+		(end 98.425 89.025)
 		(width 0.2)
 		(layer "F.Cu")
@@
 	)
 	(segment
-		(start 98.4125 89.0375)
-		(end 98.425 89.025)
+		(start 92.225 89.1375)
+		(end 92.325 89.0375)
 		(width 0.2)
 		(layer "F.Cu")
@@
 	)
 	(segment
-		(start 61.825 67.525)
-		(end 61.825 76.625)
-		(width 0.2)
-		(layer "F.Cu")
-		(net 62)
-	)
-	(segment
 		(start 66.075 63.275)
 		(end 66.695 62.655)
@@
 	)
 	(segment
-		(start 62.175 67.175)
-		(end 61.825 67.525)
+		(start 61.825 73.825)
+		(end 61.825 76.625)
 		(width 0.2)
 		(layer "F.Cu")
@@
 	)
 	(via
-		(at 62.175 67.175)
+		(at 61.825 73.825)
 		(size 0.6)
 		(drill 0.3)
@@
 	)
 	(segment
-		(start 62.175 67.175)
+		(start 61.825 73.825)
+		(end 61.825 67.525)
+		(width 0.2)
+		(layer "B.Cu")
+		(net 62)
+	)
+	(segment
+		(start 61.825 67.525)
 		(end 66.075 63.275)
 		(width 0.2)
@@
 	)
 	(segment
-		(start 60.125 68.025)
-		(end 60.125 70.725)
+		(start 60.125 70.725)
+		(end 60.225 70.825)
 		(width 0.2)
 		(layer "F.Cu")
@@
 	)
 	(segment
-		(start 60.125 70.725)
-		(end 60.225 70.825)
+		(start 61.275 66.875)
+		(end 60.125 68.025)
 		(width 0.2)
 		(layer "F.Cu")
@@
 	)
 	(segment
-		(start 64.600735 63.900735)
-		(end 64.625 63.925)
+		(start 64.625 63.925)
+		(end 68.475 63.925)
 		(width 0.2)
 		(layer "F.Cu")
@@
 	)
 	(segment
-		(start 62.125 66.025)
-		(end 60.125 68.025)
+		(start 64.600735 63.900735)
+		(end 64.625 63.925)
 		(width 0.2)
 		(layer "F.Cu")
@@
 	)
 	(segment
-		(start 64.625 63.925)
-		(end 68.475 63.925)
+		(start 60.125 68.025)
+		(end 60.125 70.725)
 		(width 0.2)
 		(layer "F.Cu")
@@
 	)
 	(via
-		(at 62.125 66.025)
+		(at 61.275 66.875)
 		(size 0.6)
 		(drill 0.3)
@@
 	)
 	(segment
-		(start 64.249265 63.900735)
-		(end 62.125 66.025)
+		(start 64.600735 63.900735)
+		(end 64.249265 63.900735)
 		(width 0.2)
 		(layer "B.Cu")
@@
 	)
 	(segment
-		(start 64.600735 63.900735)
-		(end 64.249265 63.900735)
+		(start 64.249265 63.900735)
+		(end 61.275 66.875)
 		(width 0.2)
 		(layer "B.Cu")
@@
 	)
 	(segment
-		(start 90.385 95.65)
-		(end 90.41 95.675)
+		(start 90.41 95.675)
+		(end 92.225 93.86)
 		(width 0.2)
 		(layer "F.Cu")
@@
 	)
 	(segment
-		(start 90.41 95.675)
-		(end 94.025 92.06)
+		(start 92.225 93.86)
+		(end 92.225 90.7125)
 		(width 0.2)
 		(layer "F.Cu")
@@
 	)
 	(segment
-		(start 72.78 66.13)
-		(end 72.78 65.175)
+		(start 90.385 95.65)
+		(end 90.41 95.675)
 		(width 0.2)
 		(layer "F.Cu")
@@
 	)
 	(segment
-		(start 74.475 67.825)
-		(end 72.78 66.13)
+		(start 72.78 66.13)
+		(end 72.78 65.175)
 		(width 0.2)
 		(layer "F.Cu")
@@
 	)
 	(segment
-		(start 94.025 92.06)
-		(end 94.025 90.7125)
+		(start 74.475 67.825)
+		(end 72.78 66.13)
 		(width 0.2)
 		(layer "F.Cu")
