File: DisplayDriver/DisplayDriver.kicad_sch (KiCad schematic)
At the start: 70 parts, among them J1 HTSS-108-01-G-D, J2 HEADER-1X14, J3 HTSS-108-01-G-D, SW1 (Generic) Lab Kit, U1 ESP32-S3-WROOM-1, U2 74AHCT245, U3 74AHCT245, U4 AP2112K-3.3TRG1, U5 STUSB4500QTR, X1 UJ20-C-H-G-SMT-TR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

Commit message: Major PCB Revisions.
Parts:
- removed C11, C15, C5: 0.1uF, Capacitor_SMD:C_0603_1608Metric, symbol Device:C_Small
- removed C3, C4: 10uF, Capacitor_SMD:C_0805_2012Metric_Pad1.18x1.45mm_HandSolder, symbol Adafruit MatrixPortal S3-eagle-import:CAP_CERAMIC0805-NOOUTLINE
- removed D4: ESDA25P35-1U1M, ESDA25P35-1U1M:TVS_ESDA25P35-1U1M, symbol ESDA25P35-1U1M:ESDA25P35-1U1M
- removed D5: ESDA25W, ESDA25W:SOT65P210X110-3N, symbol ESDA25W:ESDA25W
- removed PC1: 100uF/6.3V, Capacitor_SMD:C_0805_2012Metric_Pad1.18x1.45mm_HandSolder, symbol Adafruit MatrixPortal S3-eagle-import:CAP_ELECTROLYTICPANASONIC_D
- removed R23, R24: 5.1k, Resistor_SMD:R_0805_2012Metric_Pad1.20x1.40mm_HandSolder, symbol Device:R
- removed R30, R9: 4.7k, Resistor_SMD:R_0805_2012Metric_Pad1.20x1.40mm_HandSolder, symbol Device:R
- removed R31, R32: 22, Resistor_SMD:R_0805_2012Metric_Pad1.20x1.40mm_HandSolder, symbol Device:R
- removed R8: 100k, Resistor_SMD:R_0805_2012Metric_Pad1.20x1.40mm_HandSolder, symbol Device:R
- removed U4: AP2112K-3.3TRG1, DisplayDriver:SOT95P285X140-5N, symbol AP2112K-3.3TRG1:AP2112K-3.3TRG1
- removed U5: STUSB4500QTR, Package_DFN_QFN:QFN-24-1EP_4x4mm_P0.5mm_EP2.7x2.7mm, symbol Interface_USB:STUSB4500QTR
- removed X1: UJ20-C-H-G-SMT-TR, DisplayDriver:CUI_UJ20-C-H-G-SMT-TR, symbol UJ20-C-H-G-SMT-TR:UJ20-C-H-G-SMT-TR
Connections:
- net DOWN: now also U1.9 (IO16); no longer U1.38 (IO2)
- net SCL: no longer J2.3 (Pin_3), U1.23 (IO21)
- net SDA: no longer J2.4 (Pin_4), U1.7 (IO7)
- net UP: now also U1.8 (IO15); no longer U1.39 (IO1)
- no-connect marks 49 -> 39
Other:
- note added: "Caps for screen power (CURRENTLY BOARD EXCLUDED!!!!!!!!!!)"
- note removed: "Caps for screen power"
- note removed: "PD system (needs buck conv. for 8A)"
- note removed: "POWER SUPPLY: 3.3V."
- note removed: "USBC 16V, 3A Power sink (PD input)"
- note removed: "add decouplng and sensing ^"
- note removed: "dead bat sense"
- note removed: "mcu present"
- note removed: "old (5v vbus)"
- note removed: "pg 26 of datasheet"
- moved on the sheet: C10, C9, J3, PC2, R25, R26, R28, R29, X2

Commit message: random
Parts:
- R25, R26: value 10k -> 56k
Changed lines of the file:
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@@
 		(company "Aviator")
 		(comment 1 "Reminder: OE, LAT - LOW at boot, BOOT0 - HIGH at reset")
-		(comment 2 "Reminder: PD USB C support with STUSB to negotiate ~50W")
+		(comment 2 "Reminder: Configure ESP32 as host of ADSB")
 		(comment 3 "Reminder: 22-100ohm on hub75 if ringing")
 	)
@@
 			)
 		)
-		(property "Value" "10k"
+		(property "Value" "56k"
 			(at 50.292 137.16 90)
 			(effects
@@
 			)
 		)
-		(property "Value" "10k"
+		(property "Value" "56k"
 			(at 54.102 144.78 90)
 			(effects
