File: DisplayDriver/DisplayDriver.kicad_sch (KiCad schematic)
At the start: 74 parts, among them SW1 KMR2, SW2 KMR2, U1 ESP32-S3-WROOM, U10 74AHCT245, U2 74AHCT245, U3 74AHCT245, U4 AP2112K-3.3, U5 ESP32-WROVER-B, U6 CH340N, U7 CP2102N-Axx-xQFN24, U8 ESP32-WROVER-B, U9 74AHCT245, X1 USB TYPE C

Commit message: final
Connections:
- net ADDRD_3V is gone; now on net GND: U10.8 (A7), U3.4 (A3), U5.9 (IO33), U8.9 (IO33)
- net B1_3V: now also U8.31 (IO19), U9.8 (A7); no longer U8.33 (IO21), U9.7 (A6)
- net G1_3V: now also U8.33 (IO21), U9.7 (A6); no longer U8.31 (IO19), U9.8 (A7)
- net M1_A: now also JP5.6
- net M1_B: now also JP5.5
- net M1_B1: now also U9.12 (B7); no longer U9.13 (B6)
- net M1_C: now also JP5.4
- net M1_D: now also JP5.3
- net M1_G1: now also U9.13 (B6); no longer U9.12 (B7)
Other:
- moved on the sheet: C19, C21, D1, DOWN2A, JP4, JP5, L2, R11, R12, R13, R15, R16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

Commit message: PCB commit pls
Parts:
- removed C1: 0.1uF, Adafruit MatrixPortal S3:0603-NO, symbol Adafruit MatrixPortal S3-eagle-import:CAP_CERAMIC0603_NO
- removed C19: 10uF, Adafruit MatrixPortal S3:0805-NO, symbol Adafruit MatrixPortal S3-eagle-import:CAP_CERAMIC0805-NOOUTLINE
- removed C21: 1uF, Adafruit MatrixPortal S3:0603-NO, symbol Adafruit MatrixPortal S3-eagle-import:CAP_CERAMIC0603_NO
- removed D1: 3.6V, Adafruit MatrixPortal S3:SOD-323, symbol Adafruit MatrixPortal S3-eagle-import:DIODE-ZENERSOD323
- removed DOWN2, RST2, UP2: TL3330AF260QG, Adafruit MatrixPortal S3:SPST_TACTILE_RA, symbol Adafruit MatrixPortal S3-eagle-import:SWITCH_SPST_MNT_TACT_RA
- removed JP1, JP3, JP4: 2x8_SMT_IDC, Adafruit MatrixPortal S3:2X08_SHROUDEDSMT, symbol Adafruit MatrixPortal S3-eagle-import:HEADER-2X8_SHROUDEDSMT
- removed JP5: HEADER-1X11, Adafruit MatrixPortal S3:1X11_ROUND, symbol Adafruit MatrixPortal S3-eagle-import:HEADER-1X11
- removed L2: RED, Adafruit MatrixPortal S3:CHIPLED_0603_NOOUTLINE, symbol Adafruit MatrixPortal S3-eagle-import:LED0603_NOOUTLINE
- removed LED2: WS2812B_3535FULL, Adafruit MatrixPortal S3:LED3535_FULLPADS, symbol Adafruit MatrixPortal S3-eagle-import:WS2812B_3535FULL
- removed R10: 22, symbol Device:R
- removed R11, R13, R15, R16, R17: 10K, Adafruit MatrixPortal S3:0603-NO, symbol Adafruit MatrixPortal S3-eagle-import:RESISTOR_0603_NOOUT
- removed R12: 1K, Adafruit MatrixPortal S3:0603-NO, symbol Adafruit MatrixPortal S3-eagle-import:RESISTOR_0603_NOOUT
- removed SENSE1: JST PH 3, Adafruit MatrixPortal S3:JSTPH3, symbol Adafruit MatrixPortal S3-eagle-import:CON_JST_PH_3PIN
- removed SJ3: SOLDERJUMPER_2WAY, Adafruit MatrixPortal S3:SOLDERJUMPER_2WAY_OPEN_NOPASTE, symbol Adafruit MatrixPortal S3-eagle-import:SOLDERJUMPER_2WAY
- removed SW2: KMR2, Adafruit MatrixPortal S3:BTN_RKB2_4.6X2.8, symbol Adafruit MatrixPortal S3-eagle-import:SWITCH_TACT_SMT_RKB2
- removed U1: ESP32-S3-WROOM, Adafruit MatrixPortal S3:S3-WROOM32, symbol Adafruit MatrixPortal S3-eagle-import:ESP32-S3-WROOM
- removed U10, U9: 74AHCT245, Adafruit MatrixPortal S3:TSSOP20, symbol Adafruit MatrixPortal S3-eagle-import:74LCX245_TSSOP20
- removed U6: CH340N, Package_SO:SOP-8_3.9x4.9mm_P1.27mm, symbol Interface_USB:CH340N
- removed U7: CP2102N-Axx-xQFN24, Package_DFN_QFN:QFN-24-1EP_4x4mm_P0.5mm_EP2.6x2.6mm, symbol Interface_USB:CP2102N-Axx-xQFN24
- removed U8: ESP32-WROVER-B, RF_Module:ESP32-WROVER-B, symbol RF_Module:ESP32-S2-WROVER
- removed UNK3VON2, UNK5VON2: GREEN, Adafruit MatrixPortal S3:CHIPLED_0603_NOOUTLINE, symbol Adafruit MatrixPortal S3-eagle-import:LED0603_NOOUTLINE
- added J1, J3: HTSS-108-01-G-D, HTSS-108-01-G-D:SAMTEC_HTSS-108-01-G-D, symbol HTSS-108-01-G-D:HTSS-108-01-G-D
- added R2: 10K, Adafruit MatrixPortal S3:0603-NO, symbol Adafruit MatrixPortal S3-eagle-import:RESISTOR_0603_NOOUT
- added SJ2: SOLDERJUMPER_2WAY, symbol Jumper:SolderJumper_3_Open
- R9: value 22 -> 330
- renumbered JP2 to J2, U5 to U1
Connections:
- net D+ is gone; now on net NEOPIX: R9.1
- net 3.3V: now also R2.2
- net ADDRA_3V: now also U1.37 (IO23), U2.2 (A1); no longer U1.36 (IO22), U3.5 (A4)
- net ADDRB_3V: now also U1.36 (IO22), U2.3 (A2); no longer U1.37 (IO23), U2.9 (A8)
- net ADDRC_3V: now also U1.9 (IO33), U3.8 (A7); no longer U1.8 (IO32), U3.6 (A5)
- net ADDRE_3V: now also U2.7 (A6); no longer U3.8 (A7)
- net B1_3V: now also U1.31 (IO19), U2.5 (A4); no longer U1.33 (IO21), U2.4 (A3)
- net B2_3V: now also U3.5 (A4); no longer U2.7 (A6)
- net BOOT0: now also R2.1, SJ2.1 (A); no longer U1.25 (STRAP_IO0)
- net CLK: now also U3.16 (B3), J1.13, J3.13; no longer U2.12 (B7)
- net CLK_3V: now also U3.4 (A3); no longer U2.8 (A7)
- net G1_3V: now also U1.33 (IO21), U2.4 (A3); no longer U1.31 (IO19), U2.3 (A2)
- net G2_3V: now also U3.6 (A5); no longer U2.5 (A4)
- net GND: now also J1.04, J3.04; no longer U1.9 (IO33), U3.4 (A3)
- net LAT: now also U2.11 (B8), J1.14, J3.14; no longer U3.13 (B6)
- net LAT_3V: now also U2.9 (A8); no longer U3.7 (A6)
- net M1_A: now also U2.18 (B1), J1.09, J3.09; no longer U3.15 (B4)
- net M1_B: now also U2.17 (B2), J1.10, J3.10; no longer U2.11 (B8)
- net M1_B1: now also U2.15 (B4), J1.03, J3.03; no longer U2.16 (B3)
- net M1_B2: now also U3.15 (B4), J1.07, J3.07; no longer U2.13 (B6)
- net M1_C: now also U3.12 (B7), J1.11, J3.11; no longer U3.14 (B5)
- net M1_D: now also U3.11 (B8), J1.12, J3.12; no longer U3.16 (B3)
- net M1_E: now also U2.13 (B6); no longer U3.12 (B7)
- net M1_E16: now also J1.16, J3.16
- net M1_E8: now also J1.08, J3.08
- net M1_G1: now also U2.16 (B3), J1.02, J3.02; no longer U2.17 (B2)
- net M1_G2: now also U3.14 (B5), J1.06, J3.06; no longer U2.15 (B4)
- net M1_R1: now also U2.14 (B5), J1.01, J3.01; no longer U2.18 (B1)
- net M1_R2: now also U3.13 (B6), J1.05, J3.05; no longer U2.14 (B5)
- net NEOPIX: no longer LED1.1 (DI), U1.24 (STRAP_IO2)
- net OE: now also U2.12 (B7), J1.15, J3.15; no longer U3.11 (B8)
- net OE_3V: now also U2.8 (A7); no longer U3.9 (A8)
- net R1_3V: now also U2.6 (A5); no longer U2.2 (A1)
- net R2_3V: now also U3.7 (A6); no longer U2.6 (A5)
- net at R9.2: now also LED1.1 (DI)
- new net: SJ2.2 (C), U1.25 (STRAP_IO0)
- new net ADDRD_3V: U1.8 (IO32), U3.9 (A8)
- new net Neopix: U1.24 (STRAP_IO2)
Other:
- note added: "bulk ESP"
- note added: "dcpl 75HCT (2x)"
- note added: "dcpl WS28"
- note removed: "USB->Serial"
- moved on the sheet: SW1

Commit message: desktop to laptop
Parts:
- removed C15, C7: 10uF, Adafruit MatrixPortal S3:0805-NO, symbol Adafruit MatrixPortal S3-eagle-import:CAP_CERAMIC0805-NOOUTLINE
- removed C17: 0.1uF, Adafruit MatrixPortal S3:0603-NO, symbol Adafruit MatrixPortal S3-eagle-import:CAP_CERAMIC0603_NO
- removed D2: 3.6V, Adafruit MatrixPortal S3:SOD-323, symbol Adafruit MatrixPortal S3-eagle-import:DIODE-ZENERSOD323
- removed J2: HEADER-1X11, Adafruit MatrixPortal S3:1X11_ROUND, symbol Adafruit MatrixPortal S3-eagle-import:HEADER-1X11
- removed R4: 5.1K Pack, Adafruit MatrixPortal S3:RESPACK_4X0603, symbol Adafruit MatrixPortal S3-eagle-import:RESISTOR_4PACK
- removed R5: 1K, Adafruit MatrixPortal S3:0603-NO, symbol Adafruit MatrixPortal S3-eagle-import:RESISTOR_0603_NOOUT
- removed SENSE2: JST PH 3, Adafruit MatrixPortal S3:JSTPH3, symbol Adafruit MatrixPortal S3-eagle-import:CON_JST_PH_3PIN
- removed SJ2: SOLDERJUMPER_2WAY, symbol Jumper:SolderJumper_3_Open
- removed U1: ESP32-WROVER-B, RF_Module:ESP32-WROVER-B, symbol RF_Module:ESP32-S2-WROVER
- added C3: 10uF, Adafruit MatrixPortal S3:0805-NO, symbol Adafruit MatrixPortal S3-eagle-import:CAP_CERAMIC0805-NOOUTLINE
- added C7: 0.1uF, Adafruit MatrixPortal S3:0603-NO, symbol Adafruit MatrixPortal S3-eagle-import:CAP_CERAMIC0603_NO
- added J2: HEADER-1X14, symbol Connector:Conn_01x14_Pin
- added R8, R9: 5.1k, symbol Device:R
- added U1: ESP32-S3-WROOM-1, RF_Module:ESP32-S3-WROOM-1, symbol RF_Module:ESP32-S3-WROOM-1
- added U5: STUSB4500QTR, Package_DFN_QFN:QFN-24-1EP_4x4mm_P0.5mm_EP2.7x2.7mm, symbol Interface_USB:STUSB4500QTR
- renumbered R2 to R1, R1 to R2, R7 to R4, R6 to R5, R8 to R6, R9 to R7
Connections:
- net VCC is gone; now on net GND: C5.1
- net +5V: now also C3.2, J2.12 (Pin_12)
- net 3.3V: now also C5.2, C7.2, J2.13 (Pin_13), U1.2 (3V3)
- net ADDRA_3V: now also U3.5 (A4), U1.31 (IO38); no longer U2.2 (A1)
- net ADDRB_3V: now also U3.6 (A5), U1.32 (IO39); no longer U2.3 (A2)
- net ADDRC_3V: now also U3.7 (A6), U1.33 (IO40); no longer U3.8 (A7)
- net ADDRD_3V: now also U3.8 (A7), U1.34 (IO41); no longer U3.9 (A8)
- net ADDRE_3V: now also U3.9 (A8), U1.35 (IO42); no longer U2.7 (A6)
- net B1_3V: now also U2.4 (A3), U1.12 (IO8); no longer U2.5 (A4)
- net B2_3V: now also U2.7 (A6), U1.19 (IO11); no longer U3.5 (A4)
- net BOOT0: now also J2.2 (Pin_2), U1.27 (IO0)
- net CC1: now also R9.1
- net CC2: now also R8.1
- net CLK_3V: now also U1.4 (IO4)
- net DOWN: now also U1.38 (IO2)
- net G1_3V: now also U2.3 (A2), U1.7 (IO7); no longer U2.4 (A3)
- net G2_3V: now also U2.6 (A5), U1.18 (IO10); no longer U3.6 (A5)
- net GND: now also C3.1, C7.1, J2.14 (Pin_14), R8.2, R9.2, U1.1 (GND), U1.40 (GND), U1.41 (GND); no longer C5.2
- net LAT_3V: now also U1.5 (IO5)
- net M1_A: now also U3.15 (B4); no longer U2.18 (B1)
- net M1_B: now also U3.14 (B5); no longer U2.17 (B2)
- net M1_B1: now also U2.16 (B3); no longer U2.15 (B4)
- net M1_B2: now also U2.13 (B6); no longer U3.15 (B4)
- net M1_C: now also U3.13 (B6); no longer U3.12 (B7)
- net M1_D: now also U3.12 (B7); no longer U3.11 (B8)
- net M1_E: now also U3.11 (B8); no longer U2.13 (B6)
- net M1_G1: now also U2.17 (B2); no longer U2.16 (B3)
- net M1_G2: now also U2.14 (B5); no longer U3.14 (B5)
- net M1_R1: now also U2.18 (B1); no longer U2.14 (B5)
- net M1_R2: now also U2.15 (B4); no longer U3.13 (B6)
- net NEOPIX: now also J2.11 (Pin_11), U1.26 (IO45)
- net OE_3V: now also U1.15 (IO3); no longer R3.2
- net R1_3V: now also U2.2 (A1), U1.6 (IO6); no longer U2.6 (A5)
- net R2_3V: now also U2.5 (A4), U1.17 (IO9); no longer U3.7 (A6)
- net UP: now also U1.39 (IO1)
- net ~{RESET}: now also J2.1 (Pin_1), U1.3 (EN)
- net D+ (NC) renamed D+
- net D+: now also U1.14 (IO20)
- net D- (NC) renamed D-
- net D-: now also U1.13 (IO19)
- net D15 renamed D13
- net D13: now also U1.21 (IO13)
- new net: U5.10 (GND), U5.25 (GND)
- new net I2C_SCL: J2.10 (Pin_10), U1.11 (IO18)
- new net I2C_SDA: J2.9 (Pin_9), U1.10 (IO17)
- new net NC: U1.20 (IO12)
- new net NC1: U1.8 (IO15)
- new net NC2: U1.9 (IO16)
- new net NC3: U1.16 (IO46)
- new net NC4: U1.30 (IO37)
- new net NC5: U1.29 (IO36)
- new net NC6: U1.28 (IO35)
- new net SPI_CS: J2.7 (Pin_7), U1.24 (IO47)
- new net SPI_MISO: J2.5 (Pin_5), U1.22 (IO14)
- new net SPI_MOSI: J2.8 (Pin_8), U1.25 (IO48)
- new net SPI_SCLK: J2.6 (Pin_6), U1.23 (IO21)
- new net UART_RX: J2.3 (Pin_3), U1.36 (RXD0)
- new net UART_TX: J2.4 (Pin_4), U1.37 (TXD0)
- no-connect marks 0 -> 9
Other:
- note added: "ESP 32 S3 WROOM 1"
- note added: "POWER & D13 LEDS"
- note removed: "ESP32 S2 WROVER"
- note removed: "JST PH"
- note removed: "POWER & D15 LEDS"
- moved on the sheet: C10, C11, C12, C13, C14, C16, C18, C20, C4, C6, C8, C9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

Commit message: eod lab thurs
Parts:
- added J4: USB3_A, symbol Connector:USB3_A
Connections:
- net ADDRA_3V: now also U3.9 (A8); no longer U3.5 (A4)
- net ADDRB_3V: now also U3.8 (A7); no longer U3.6 (A5)
- net ADDRD_3V: now also U3.6 (A5); no longer U3.8 (A7)
- net ADDRE_3V: now also U3.5 (A4); no longer U3.9 (A8)
- net G1_3V: now also U1.11 (IO18); no longer U1.7 (IO7)
- net I2C_SCL: no longer U1.11 (IO18)
- net I2C_SDA: no longer U1.10 (IO17)
- net LAT_3V: now also U1.20 (IO12); no longer U1.5 (IO5)
- net M1_A: now also U3.11 (B8); no longer U3.15 (B4)
- net M1_B: now also U3.12 (B7); no longer U3.14 (B5)
- net M1_D: now also U3.14 (B5); no longer U3.12 (B7)
- net M1_E: now also U3.15 (B4); no longer U3.11 (B8)
- net NC: now also U1.5 (IO5); no longer U1.20 (IO12)
- net NC3: now also U1.25 (IO48); no longer U1.16 (IO46)
- net NC4: now also U1.24 (IO47); no longer U1.30 (IO37)
- net NC5: now also U1.16 (IO46); no longer U1.29 (IO36)
- net NC6: now also U1.30 (IO37); no longer U1.28 (IO35)
- net R1_3V: now also U1.10 (IO17); no longer U1.6 (IO6)
- net SPI_CS: no longer U1.24 (IO47)
- net SPI_MISO: no longer U1.22 (IO14)
- net SPI_MOSI: no longer U1.25 (IO48)
- net SPI_SCLK: no longer U1.23 (IO21)
- new net NC7: U1.29 (IO36)
- new net NC8: U1.28 (IO35)
Other:
- note added: "ADSB USB3A"

Commit message: halfway commit PCB
Parts:
- removed C10, C5, C6: 10uF, Adafruit MatrixPortal S3:0805-NO, symbol Adafruit MatrixPortal S3-eagle-import:CAP_CERAMIC0805-NOOUTLINE
- removed C14, C20, C8: 0.1uF, Adafruit MatrixPortal S3:0603-NO, symbol Adafruit MatrixPortal S3-eagle-import:CAP_CERAMIC0603_NO
- removed C4: 1uF, Adafruit MatrixPortal S3:0603-NO, symbol Adafruit MatrixPortal S3-eagle-import:CAP_CERAMIC0603_NO
- removed J4: USB3_A, symbol Connector:USB3_A
- removed R8, R9: 5.1k, symbol Device:R
- removed U4: AP2112K-3.3, Adafruit MatrixPortal S3:SOT23-DBV, symbol Adafruit MatrixPortal S3-eagle-import:LP2985-XXDBVR
- removed X1: USB TYPE C, Adafruit MatrixPortal S3:USB_C_CUSB31-CFM2AX-01-X, symbol Adafruit MatrixPortal S3-eagle-import:USB_C
- added C1.1, C3.1: 10uF, Adafruit MatrixPortal S3:0805-NO, symbol Adafruit MatrixPortal S3-eagle-import:CAP_CERAMIC0805-NOOUTLINE
- added C10, C15, C16, C5: 0.1uF, Capacitor_SMD:C_0805_2012Metric_Pad1.18x1.45mm_HandSolder, symbol Adafruit MatrixPortal S3-eagle-import:CAP_CERAMIC0603_NO
- added C14, C4, C8: 10uF, Capacitor_SMD:C_0805_2012Metric_Pad1.18x1.45mm_HandSolder, symbol Adafruit MatrixPortal S3-eagle-import:CAP_CERAMIC0805-NOOUTLINE
- added C5.1: 0.1uF, Adafruit MatrixPortal S3:0603-NO, symbol Adafruit MatrixPortal S3-eagle-import:CAP_CERAMIC0603_NO
- added PC1.1: 100uF/6.3V, Adafruit MatrixPortal S3:PANASONIC_D, symbol Adafruit MatrixPortal S3-eagle-import:CAP_ELECTROLYTICPANASONIC_D
- added R8: 5.1k, Resistor_SMD:R_0805_2012Metric_Pad1.20x1.40mm_HandSolder, symbol Adafruit MatrixPortal S3-eagle-import:RESISTOR_4PACK
- added R8A.1, R8B.1: 5.1k, symbol Device:R
- added R9: 22, Resistor_SMD:R_0805_2012Metric_Pad1.20x1.40mm_HandSolder, symbol Adafruit MatrixPortal S3-eagle-import:RESISTOR_4PACK
- added U4: AP2112K-3.3TRG1, DisplayDriver:SOT95P285X140-5N, symbol AP2112K-3.3TRG1:AP2112K-3.3TRG1
- added U4.1: AP2112K-3.3, Adafruit MatrixPortal S3:SOT23-DBV, symbol Adafruit MatrixPortal S3-eagle-import:LP2985-XXDBVR
- added X1, X2: UJ20-C-H-G-SMT-TR, UJ20-C-H-G-SMT-TR:CUI_UJ20-C-H-G-SMT-TR, symbol UJ20-C-H-G-SMT-TR:UJ20-C-H-G-SMT-TR
- added X1.1: USB TYPE C, Adafruit MatrixPortal S3:USB_C_CUSB31-CFM2AX-01-X, symbol Adafruit MatrixPortal S3-eagle-import:USB_C
- C1: renamed from C16; footprint Adafruit MatrixPortal S3:0603-NO -> Capacitor_SMD:C_0805_2012Metric_Pad1.18x1.45mm_HandSolder
- C11, C12, C13, C3: footprint Adafruit MatrixPortal S3:0805-NO -> Capacitor_SMD:C_0805_2012Metric_Pad1.18x1.45mm_HandSolder
- C2: renamed from C18; footprint Adafruit MatrixPortal S3:0805-NO -> Capacitor_SMD:C_0805_2012Metric_Pad1.18x1.45mm_HandSolder
- C6: renamed from C2; footprint Adafruit MatrixPortal S3:0603-NO -> Capacitor_SMD:C_0805_2012Metric_Pad1.18x1.45mm_HandSolder
- C7: value 0.1uF -> 1uF; footprint Adafruit MatrixPortal S3:0603-NO -> Capacitor_SMD:C_0805_2012Metric_Pad1.18x1.45mm_HandSolder
- C9: footprint Adafruit MatrixPortal S3:0603-NO -> Capacitor_SMD:C_0805_2012Metric_Pad1.18x1.45mm_HandSolder
- L1: footprint Adafruit MatrixPortal S3:CHIPLED_0603_NOOUTLINE -> LED_SMD:LED_0603_1608Metric
- L2: renamed from UNK5VON1; footprint Adafruit MatrixPortal S3:CHIPLED_0603_NOOUTLINE -> LED_SMD:LED_0603_1608Metric
- L3: renamed from UNK3VON1; footprint Adafruit MatrixPortal S3:CHIPLED_0603_NOOUTLINE -> LED_SMD:LED_0603_1608Metric
- PC1: footprint Adafruit MatrixPortal S3:PANASONIC_D -> Capacitor_SMD:C_0805_2012Metric_Pad1.18x1.45mm_HandSolder
- R1, R2, R3, R4, R5, R6: footprint Adafruit MatrixPortal S3:0603-NO -> Resistor_SMD:R_0805_2012Metric_Pad1.20x1.40mm_HandSolder
- R7: value 330 -> Resistor_SMD:R_0805_2012Metric_Pad1.20x1.40mm_HandSolder; footprint (none) -> Resistor_SMD:R_0805_2012Metric_Pad1.20x1.40mm_HandSolder
- SW1: value KMR2 -> Generic (Lab Kit); footprint Adafruit MatrixPortal S3:BTN_RKB2_4.6X2.8 -> Button_Switch_THT:SW_PUSH_6mm
Connections:
- net +5V: now also U4.1 (VIN), U4.1.1 (IN), U4.1.3 (ON/~{OFF}), U4.3 (EN), X1.A4 (VBUS), X1.A9 (VBUS), X1.B4 (VBUS), X1.B9 (VBUS)
- net 3.3V: now also C7.1, C1.1.2, C10.2, C14.1, C15.2, C16.1, C4.2, C5.1.2, C5.2, C8.1, U4.1.5 (OUT), U4.5 (VOUT); no longer C7.2
- net B1_3V: now also U1.17 (IO9), U2.5 (A4); no longer U1.12 (IO8), U2.4 (A3)
- net B2_3V: now also U1.11 (IO18), U2.8 (A7); no longer U1.19 (IO11), U2.7 (A6)
- net CC1: now also R8.7 (2), X1.A5 (CC1)
- net CC2: now also R8.8 (2), X1.B5 (CC2)
- net G1_3V: now also U1.18 (IO10), U2.4 (A3); no longer U1.11 (IO18), U2.3 (A2)
- net G2_3V: now also U1.12 (IO8), U2.7 (A6); no longer U1.18 (IO10), U2.6 (A5)
- net GND: now also C7.2, C1.1.1, C10.1, C14.2, C15.1, C16.2, C3.1.1, C4.1, C5.1, C5.1.1, C8.2, PC1.1.-, R8.1, R8.2 (1), R8.3 (1), R8.4 (1), R8A.1.2, R8B.1.2, U4.1.2 (GND), U4.2 (GND), X1.1.A1B12 (GND), X1.1.B1A12 (GND), X1.A1 (GND), X1.A12 (GND), X1.B1 (GND), X1.B12 (GND), X1.SH1 (SHIELD), X1.SH2 (SHIELD), X1.SH3 (SHIELD), X1.SH4 (SHIELD), X2.A1 (GND), X2.A12 (GND), X2.B1 (GND), X2.B12 (GND), X2.SH1 (SHIELD), X2.SH2 (SHIELD), X2.SH3 (SHIELD), X2.SH4 (SHIELD); no longer C7.1
- net LAT: now also U2.18 (B1); no longer U2.11 (B8)
- net LAT_3V: now also U2.2 (A1); no longer U2.9 (A8)
- net M1_B1: now also U2.15 (B4); no longer U2.16 (B3)
- net M1_B2: now also U2.12 (B7); no longer U2.13 (B6)
- net M1_G1: now also U2.16 (B3); no longer U2.17 (B2)
- net M1_G2: now also U2.13 (B6); no longer U2.14 (B5)
- net M1_R1: now also U2.17 (B2); no longer U2.18 (B1)
- net M1_R2: now also U2.14 (B5); no longer U2.15 (B4)
- net NC1: now also U1.6 (IO6); no longer U1.8 (IO15)
- net NC2: now also U1.7 (IO7); no longer U1.9 (IO16)
- net NC3: now also U1.22 (IO14); no longer U1.25 (IO48)
- net NC4: now also U1.8 (IO15); no longer U1.24 (IO47)
- net NC5: now also U1.9 (IO16); no longer U1.16 (IO46)
- net NC6: now also U1.25 (IO48); no longer U1.30 (IO37)
- net NC7: now also U1.24 (IO47); no longer U1.29 (IO36)
- net NC8: now also U1.16 (IO46); no longer U1.28 (IO35)
- net OE: now also U2.11 (B8); no longer U2.12 (B7)
- net OE_3V: now also U1.10 (IO17), U2.9 (A8); no longer U1.15 (IO3), U2.8 (A7)
- net R1_3V: now also U1.19 (IO11), U2.3 (A2); no longer U1.10 (IO17), U2.2 (A1)
- net R2_3V: now also U1.15 (IO3), U2.6 (A5); no longer U1.17 (IO9), U2.5 (A4)
- net NC9: now reaches U1.23 (IO21)
- net D+ renamed D1+
- net D1+: now also R9.7 (2)
- net D- renamed D1-
- net D1-: now also R9.8 (2)
- net I2C_SCL: no longer names the net of J2.10 (Pin_10)
- net I2C_SDA: no longer names the net of J2.9 (Pin_9)
- net SPI_CS: no longer names the net of J2.7 (Pin_7)
- net SPI_MISO: no longer names the net of J2.5 (Pin_5)
- net SPI_MOSI: no longer names the net of J2.8 (Pin_8)
- net SPI_SCLK: no longer names the net of J2.6 (Pin_6)
- new net: R9.2 (1), X1.A6 (DP1), X1.B6 (DP2)
- new net: R9.1, X1.A7 (DN1), X1.B7 (DN2)
- new net: R9.4 (1), X2.A6 (DP1), X2.B6 (DP2)
- new net: X2.A4 (VBUS), X2.A9 (VBUS), X2.B4 (VBUS), X2.B9 (VBUS)
- new net: R9.3 (1), X2.A7 (DN1), X2.B7 (DN2)
- new net +5V.: C3.1.2, PC1.1.+, X1.1.A4B9 (VBUS), X1.1.B4A9 (VBUS)
- new net CC1.: R8B.1.1, X1.1.A5 (CC1)
- new net CC1A: R8.5 (2), X2.A5 (CC1)
- new net CC2.: R8A.1.1, X1.1.B5 (CC2)
- new net CC2A: R8.6 (2), X2.B5 (CC2)
- new net D1+.: X1.1.A6 (D+), X1.1.B6 (D+)
- new net D1-.: X1.1.A7 (D-), X1.1.B7 (D-)
- new net D2+: R9.5 (2)
- new net D2-: R9.6 (2)
- no-connect marks 9 -> 29
Other:
- note added: "ADSB USBC"
- note added: "USBC 5A,5V Power"
- note removed: "ADSB USB3A"
- note removed: "USB Connection & Power."
- moved on the sheet: R3

Commit message: pcb
Parts:
- removed C1.1, C3.1: 10uF, Adafruit MatrixPortal S3:0805-NO, symbol Adafruit MatrixPortal S3-eagle-import:CAP_CERAMIC0805-NOOUTLINE
- removed C5.1: 0.1uF, Adafruit MatrixPortal S3:0603-NO, symbol Adafruit MatrixPortal S3-eagle-import:CAP_CERAMIC0603_NO
- removed PC1.1: 100uF/6.3V, Adafruit MatrixPortal S3:PANASONIC_D, symbol Adafruit MatrixPortal S3-eagle-import:CAP_ELECTROLYTICPANASONIC_D
- removed R8A.1, R8B.1: 5.1k, symbol Device:R
- removed U4.1: AP2112K-3.3, Adafruit MatrixPortal S3:SOT23-DBV, symbol Adafruit MatrixPortal S3-eagle-import:LP2985-XXDBVR
- removed X1.1: USB TYPE C, Adafruit MatrixPortal S3:USB_C_CUSB31-CFM2AX-01-X, symbol Adafruit MatrixPortal S3-eagle-import:USB_C
- J1: footprint HTSS-108-01-G-D:SAMTEC_HTSS-108-01-G-D -> Connector_IDC:IDC-Header_2x08_P2.54mm_Vertical
- U2, U3: footprint Adafruit MatrixPortal S3:TSSOP20 -> Package_SO:SOIC-20W_7.5x12.8mm_P1.27mm
Connections:
- no-connect marks 29 -> 26
