File: DisplayDriver/DisplayDriver.kicad_sch (KiCad schematic)
At the start: 45 parts, among them J1 HTSS-108-01-G-D, J2 HEADER-1X14, J3 HTSS-108-01-G-D, SW1 Generic (Lab Kit), U1 ESP32-S3-WROOM-1, U2 74AHCT245, U3 74AHCT245, U4 AP2112K-3.3TRG1, U5 STUSB4500QTR, X1 UJ20-C-H-G-SMT-TR, X2 UJ20-C-H-G-SMT-TR

Commit message: PCB wiring
Parts:
- removed C1, C10, C15, C16, C5, C9: 0.1uF, Capacitor_SMD:C_0805_2012Metric_Pad1.18x1.45mm_HandSolder, symbol Adafruit MatrixPortal S3-eagle-import:CAP_CERAMIC0603_NO
- removed C11, C12, C2: 10uF, Capacitor_SMD:C_0805_2012Metric_Pad1.18x1.45mm_HandSolder, symbol Adafruit MatrixPortal S3-eagle-import:CAP_CERAMIC0805-NOOUTLINE
- removed L1: RED, LED_SMD:LED_0603_1608Metric, symbol Adafruit MatrixPortal S3-eagle-import:LED0603_NOOUTLINE
- removed L2, L3: GREEN, LED_SMD:LED_0603_1608Metric, symbol Adafruit MatrixPortal S3-eagle-import:LED0603_NOOUTLINE
- removed R3: 10K, Resistor_SMD:R_0805_2012Metric_Pad1.20x1.40mm_HandSolder, symbol Adafruit MatrixPortal S3-eagle-import:RESISTOR_0603_NOOUT
- removed R8: 5.1k, Resistor_SMD:R_0805_2012Metric_Pad1.20x1.40mm_HandSolder, symbol Adafruit MatrixPortal S3-eagle-import:RESISTOR_4PACK
- removed R9: 22, Resistor_SMD:R_0805_2012Metric_Pad1.20x1.40mm_HandSolder, symbol Adafruit MatrixPortal S3-eagle-import:RESISTOR_4PACK
- removed SW1: Generic (Lab Kit), Button_Switch_THT:SW_PUSH_6mm, symbol Adafruit MatrixPortal S3-eagle-import:SWITCH_TACT_SMT_RKB2
- added C1, C15, C16, C17, C2, C5: 0.1uF, Capacitor_SMD:C_0603_1608Metric, symbol Device:C_Small
- added C10, C9: 100uF, Capacitor_SMD:C_0805_2012Metric_Pad1.18x1.45mm_HandSolder, symbol Adafruit MatrixPortal S3-eagle-import:CAP_CERAMIC0805-NOOUTLINE
- added D1: RED, LED_SMD:LED_0603_1608Metric, symbol Device:LED
- added D2, D3: GREEN, LED_SMD:LED_0603_1608Metric, symbol Device:LED
- added PC2: 1000uF/6.3V, Capacitor_SMD:C_0805_2012Metric_Pad1.18x1.45mm_HandSolder, symbol Adafruit MatrixPortal S3-eagle-import:CAP_ELECTROLYTICPANASONIC_D
- added R10, R11: 33, Resistor_SMD:R_0805_2012Metric_Pad1.20x1.40mm_HandSolder, symbol Device:R
- added R12, R13, R14, R15, R16, R17, R18, R19, R20, R21, R22: 22, Resistor_SMD:R_0603_1608Metric, symbol Device:R
- added R23, R24, R25, R26: 5.1k, Resistor_SMD:R_0805_2012Metric_Pad1.20x1.40mm_HandSolder, symbol Device:R
- added R27, R28, R29, R8: 22, Resistor_SMD:R_0805_2012Metric_Pad1.20x1.40mm_HandSolder, symbol Device:R
- added R3: 33, Resistor_SMD:R_0603_1608Metric, symbol Device:R
- added SW1: (Generic) Lab Kit, Button_Switch_THT:SW_PUSH_6mm, symbol Switch:SW_Push
- C13: value 10uF -> 100uF
- DOWN1, RST1, UP1: footprint Adafruit MatrixPortal S3:SPST_TACTILE_RA -> DisplayDriver:SW_TL3330AF260QG
- J2: footprint (none) -> Connector_PinHeader_2.54mm:PinHeader_1x14_P2.54mm_Vertical
- LED1: footprint Adafruit MatrixPortal S3:LED3535_FULLPADS -> LED_SMD:LED_WS2812B_PLCC4_5.0x5.0mm_P3.2mm
- R7: value Resistor_SMD:R_0805_2012Metric_Pad1.20x1.40mm_HandSolder -> 330
Connections:
- net CC1 is gone; now on net CC1A: X1.A5 (CC1)
- net CC2 is gone; now on net CC2A: X1.B5 (CC2)
- net +5V: now also C14.2, C1.1, C10.2, C15.1, C2.1, C9.2, PC2.+
- net 3.3V: now also C13.2, C7.2, C8.2, C16.1, C17.1, C5.1, D3.2 (A); no longer C13.1, C14.1, C7.1, C8.1
- net BOOT0: now also SW1.1
- net CC1A: now also R24.1; no longer X2.A5 (CC1)
- net CC2A: now also R23.1; no longer X2.B5 (CC2)
- net CLK_3V: now also R3.1; no longer U3.4 (A3)
- net D13: now also D1.2 (A)
- net GND: now also C13.1, C14.1, C7.1, C8.1, C1.2, C10.1, C15.2, C16.2, C17.2, C2.2, C5.2, C9.1, D2.1 (K), PC2.-, R23.2, R24.2, R25.2, R26.2, SW1.2; no longer C13.2, C14.2, C7.2, C8.2
- net LAT_3V: now also R11.1; no longer U2.2 (A1)
- net M1_A: now also R22.2; no longer U3.11 (B8)
- net M1_B: now also R21.2; no longer U3.12 (B7)
- net M1_B1: now also R14.2; no longer U2.15 (B4)
- net M1_B2: now also R17.2; no longer U2.12 (B7)
- net M1_C: now also R20.2; no longer U3.13 (B6)
- net M1_D: now also R19.2; no longer U3.14 (B5)
- net M1_E: now also R18.2; no longer U3.15 (B4)
- net M1_G1: now also R13.2; no longer U2.16 (B3)
- net M1_G2: now also R16.2; no longer U2.13 (B6)
- net M1_R1: now also R12.2; no longer U2.17 (B2)
- net M1_R2: now also R15.2; no longer U2.14 (B5)
- net OE_3V: now also R10.1; no longer U2.9 (A8)
- net DP_A: now reaches X1.A6 (DP1), X1.B6 (DP2)
- net DP_A: now also R27.1
- net at R5.1: now also D3.1 (K)
- net DN_A: now reaches X1.A7 (DN1), X1.B7 (DN2)
- net DN_A: now also R8.1
- net at R4.2: now also D2.2 (A)
- net at R6.1: now also D1.1 (K)
- net DP_B: now reaches X2.A6 (DP1), X2.B6 (DP2)
- net DP_B: now also R29.1
- net DN_B: now reaches X2.A7 (DN1), X2.B7 (DN2)
- net DN_B: now also R28.1
- net D1+ renamed DA+
- net DA+: now also R27.2
- net D1- renamed DA-
- net DA-: now also R8.2
- new net: R13.1, U2.16 (B3)
- new net: R14.1, U2.15 (B4)
- new net: R22.1, U3.11 (B8)
- new net: R16.1, U2.13 (B6)
- new net: R3.2, U3.4 (A3)
- new net: R17.1, U2.12 (B7)
- new net: R10.2, U2.9 (A8)
- new net: R18.1, U3.15 (B4)
- new net: R15.1, U2.14 (B5)
- new net: R12.1, U2.17 (B2)
- new net: R11.2, U2.2 (A1)
- new net: R20.1, U3.13 (B6)
- new net: R19.1, U3.14 (B5)
- new net: R21.1, U3.12 (B7)
- new net CC1B: R26.1, X2.A5 (CC1)
- new net CC2B: R25.1, X2.B5 (CC2)
- new net DB+: R29.2
- new net DB-: R28.2
- no-connect marks 26 -> 50
Other:
- note added: "STUSB (add caps if using)"
- note removed: "dcpl WS28"
- moved on the sheet: C13, C14, C7, C8, R7, U1

Commit message: aaa
aa
Parts:
- removed C15, C5: 0.1uF, Capacitor_SMD:C_0603_1608Metric, symbol Device:C_Small
- removed C3, C4: 10uF, Capacitor_SMD:C_0805_2012Metric_Pad1.18x1.45mm_HandSolder, symbol Adafruit MatrixPortal S3-eagle-import:CAP_CERAMIC0805-NOOUTLINE
- removed unit 2 of DOWN1
- removed PC1: 100uF/6.3V, Capacitor_SMD:C_0805_2012Metric_Pad1.18x1.45mm_HandSolder, symbol Adafruit MatrixPortal S3-eagle-import:CAP_ELECTROLYTICPANASONIC_D
- removed R23, R24: 5.1k, Resistor_SMD:R_0805_2012Metric_Pad1.20x1.40mm_HandSolder, symbol Device:R
- removed R27, R8: 22, Resistor_SMD:R_0805_2012Metric_Pad1.20x1.40mm_HandSolder, symbol Device:R
- removed unit 2 of RST1
- removed U4: AP2112K-3.3TRG1, DisplayDriver:SOT95P285X140-5N, symbol AP2112K-3.3TRG1:AP2112K-3.3TRG1
- removed U5: STUSB4500QTR, Package_DFN_QFN:QFN-24-1EP_4x4mm_P0.5mm_EP2.7x2.7mm, symbol Interface_USB:STUSB4500QTR
- removed unit 2 of UP1
- removed X1: UJ20-C-H-G-SMT-TR, UJ20-C-H-G-SMT-TR:CUI_UJ20-C-H-G-SMT-TR, symbol UJ20-C-H-G-SMT-TR:UJ20-C-H-G-SMT-TR
- J1: footprint Connector_IDC:IDC-Header_2x08_P2.54mm_Vertical -> DisplayDriver:IDC-Header_2x08_P2.54mm_Vertical
- J3: footprint HTSS-108-01-G-D:SAMTEC_HTSS-108-01-G-D -> Connector_IDC:IDC-Header_2x08_P2.54mm_Vertical
- R25, R26: value 5.1k -> 56k
- SJ1: footprint Adafruit MatrixPortal S3:SOLDERJUMPER_2WAY_OPEN_NOPASTE -> Jumper:SolderJumper-3_P1.3mm_Open_RoundedPad1.0x1.5mm_NumberLabels
- X2: footprint UJ20-C-H-G-SMT-TR:CUI_UJ20-C-H-G-SMT-TR -> DisplayDriver:CUI_UJ20-C-H-G-SMT-TR
Connections:
- net DA+ is gone; now on net DB+: U1.14 (IO20)
- net DA- is gone; now on net DB-: U1.13 (IO19)
- net NC is gone; now on net R2_3V: U1.5 (IO5)
- net NC4 is gone; now on net UP: U1.8 (IO15)
- net NC5 is gone; now on net DOWN: U1.9 (IO16)
- net +5V: now also R25.2, R26.1
- net CC1B: now also R26.2; no longer R26.1
- net CLK: no longer J3.13
- net D13: now also J2.10 (Pin_10)
- net DOWN: no longer U1.38 (IO2)
- net GND: no longer J3.04, R25.2, R26.2
- net LAT: no longer J3.14
- net M1_A: no longer J3.09
- net M1_B: no longer J3.10
- net M1_B1: no longer J3.03
- net M1_B2: no longer J3.07
- net M1_C: no longer J3.11
- net M1_D: no longer J3.12
- net M1_E16: no longer J3.16
- net M1_E8: no longer J3.08
- net M1_G1: no longer J3.02
- net M1_G2: no longer J3.06
- net M1_R1: no longer J3.01
- net M1_R2: no longer J3.05
- net OE: no longer J3.15
- net R2_3V: no longer U1.15 (IO3)
- net UART_RX: now also J2.5 (Pin_5); no longer J2.3 (Pin_3)
- net UART_TX: now also J2.6 (Pin_6); no longer J2.4 (Pin_4)
- net UP: no longer U1.39 (IO1)
- net NC1: no longer names the net of U1.6 (IO6)
- net NC2: no longer names the net of U1.7 (IO7)
- net NC3: no longer names the net of U1.22 (IO14)
- net NC6: no longer names the net of U1.25 (IO48)
- net NC7: no longer names the net of U1.24 (IO47)
- net NC8: no longer names the net of U1.16 (IO46)
- net NC9: no longer names the net of U1.23 (IO21)
- no-connect marks 50 -> 39
Other:
- note added: "*"
- note added: "*default strap pin"
- note added: "Caps for screen power (CURRENTLY BOARD EXCLUDED!!!!!!!!!!)"
- note added: "TO DO:"
- note added: "USBC - ADSB host (ADSB to ESP32)"
- note added: "spare for debug (if space on board)"
- note added: "will move floating caps here when final"
- note removed: "ADSB USBC"
- note removed: "POWER SUPPLY: 3.3V."
- note removed: "STUSB (add caps if using)"
- note removed: "USBC 5A,5V Power"
- note removed: "spare for debug"
- moved on the sheet: DOWN1A, J3, R25, R26, R28, R29, UP1A, X2
