File: DisplayDriver/DisplayDriver.kicad_sch (KiCad schematic)
At the start: 57 parts, among them J1 HTSS-108-01-G-D, J2 HEADER-1X14, J3 HTSS-108-01-G-D, J4 Barrel_Jack, U1 ESP32-S3-WROOM-1, U2 74AHCT245, U3 74AHCT245, U4 MCP1727-3302xSN, X2 UJ20-C-H-G-SMT-TR

Commit message: lap to PC
Parts:
- removed C3: C, symbol Device:C
- removed R8: R, symbol DisplayLibrary(sketch):R
- removed U4: MCP1727-3302xSN, Package_SO:SOIC-8_3.9x4.9mm_P1.27mm, symbol Regulator_Linear:MCP1727-3302xSN
- added C4, C5: C, symbol Device:C
- added U4: AMS1117-3.3, Package_TO_SOT_SMD:SOT-223-3_TabPin2, symbol Regulator_Linear:AMS1117-3.3
- RST1: renamed from DOWN2; value SW_Push -> (Generic) Lab Kit; footprint Connector_Molex:Molex_KK-254_AE-6410-02A_1x02_P2.54mm_Vertical -> Button_Switch_THT:SW_PUSH_6mm
Connections:
- net +5V: now also C4.1, U4.3 (VI)
- net 3.3V: now also C5.1, U4.2 (VO)
- net GND: now also C4.2, C5.2, U4.1 (GND)
- no-connect marks 29 -> 28
Other:
- note added: "Caps for screen power"
- note added: "TO DO: (this is all board exluded!)"
- note removed: "Caps for screen power (CURRENTLY BOARD EXCLUDED!!!!!!!!!!)"
- note removed: "TO DO:"

Commit message: change the ****** shifter footprint
Parts:
- removed C5: C, symbol Device:C
- removed R10, R11: 33, Resistor_SMD:R_0805_2012Metric_Pad1.20x1.40mm_HandSolder, symbol DisplayLibrary(sketch):R
- removed R12, R13, R14, R15, R16, R17, R18, R19, R20, R21, R22: 22, Resistor_SMD:R_0603_1608Metric, symbol DisplayLibrary(sketch):R
- removed R3: 33, Resistor_SMD:R_0603_1608Metric, symbol DisplayLibrary(sketch):R
- removed SJ1: SOLDERJUMPER_2WAY, Jumper:SolderJumper-3_P1.3mm_Open_RoundedPad1.0x1.5mm_NumberLabels, symbol DisplayLibrary(sketch):SOLDERJUMPER_2WAY
- added J4: Molex, Connector_Molex:Molex_KK-254_AE-6410-02A_1x02_P2.54mm_Vertical, symbol Connector:Conn_01x02_Pin
- added R8, R9: R, Resistor_SMD:R_0603_1608Metric, symbol DisplayLibrary(sketch):R
- C4: footprint (none) -> Capacitor_SMD:C_0805_2012Metric_Pad1.18x1.45mm_HandSolder
- LED1: footprint Adafruit MatrixPortal S3:LED3535_FULLPADS -> LED_SMD:LED_WS2812B_PLCC4_5.0x5.0mm_P3.2mm
- U2, U3: footprint Adafruit MatrixPortal S3:TSSOP20 -> DisplayDriver:PW20
- renumbered J4 to 5Vin1
Connections:
- net ADDRE_3V is gone; now on net G2_3V: U1.35 (IO42), U3.5 (A4)
- net M1_E16 is gone; now on net GND: J1.16, J3.16
- net M1_E8 is gone; now on net GND: J1.08, J3.08
- net +5V: now also J2.13 (Pin_13), J4.1 (Pin_1); no longer J2.12 (Pin_12)
- net 3.3V: now also J2.12 (Pin_12), R8.1; no longer J2.13 (Pin_13)
- net ADDRA_3V: now also U1.19 (IO11), U2.3 (A2); no longer U1.31 (IO38), U3.9 (A8)
- net ADDRB_3V: now also U1.18 (IO10), U2.4 (A3); no longer U1.32 (IO39), U3.8 (A7)
- net ADDRC_3V: now also U1.17 (IO9), U2.5 (A4); no longer U1.33 (IO40), U3.7 (A6)
- net ADDRD_3V: now also U1.5 (IO5), U2.6 (A5); no longer U1.34 (IO41), U3.6 (A5)
- net B1_3V: now also U1.33 (IO40), U3.7 (A6); no longer U1.17 (IO9), U2.5 (A4)
- net B2_3V: now also U1.20 (IO12), U2.2 (A1); no longer U1.11 (IO18), U2.8 (A7)
- net CLK: now also U2.13 (B6); no longer U3.16 (B3)
- net CLK_3V: now also U1.12 (IO8), U2.7 (A6); no longer U1.4 (IO4)
- net D13: now also J2.5 (Pin_5); no longer J2.10 (Pin_10)
- net G1_3V: now also U1.32 (IO39), U3.8 (A7); no longer U1.18 (IO10), U2.4 (A3)
- net G2_3V: no longer U1.12 (IO8), U2.7 (A6)
- net GND: now also U3.4 (A3), J4.2 (Pin_2), R9.2; no longer U4.1 (GND)
- net LAT: now also U2.12 (B7); no longer U2.18 (B1)
- net LAT_3V: now also U1.11 (IO18), U2.8 (A7); no longer U1.20 (IO12)
- net M1_A: now also U2.17 (B2)
- net M1_B: now also U2.16 (B3)
- net M1_B1: now also U3.13 (B6)
- net M1_B2: now also U2.18 (B1)
- net M1_C: now also U2.15 (B4)
- net M1_D: now also U2.14 (B5)
- net M1_G1: now also U3.12 (B7)
- net M1_G2: now also U3.15 (B4)
- net M1_R1: now also U3.11 (B8)
- net M1_R2: now also U3.14 (B5)
- net NEOPIX: now also J2.6 (Pin_6); no longer J2.11 (Pin_11)
- net OE_3V: now also U2.9 (A8)
- net R1_3V: now also U1.31 (IO38), U3.9 (A8); no longer U1.19 (IO11), U2.3 (A2)
- net R2_3V: now also U1.34 (IO41), U3.6 (A5); no longer U1.5 (IO5), U2.6 (A5)
- net UART_RX: now also J2.3 (Pin_3); no longer J2.5 (Pin_5)
- net UART_TX: now also J2.4 (Pin_4); no longer J2.6 (Pin_6)
- new net: R8.2, R9.1, U4.1 (GND)
- no-connect marks 28 -> 29
Other:
- moved on the sheet: C4

Commit message: lap to PC
Parts:
- removed R8, R9: R, Resistor_SMD:R_0603_1608Metric, symbol DisplayLibrary(sketch):R
- added C11: C, Capacitor_SMD:C_0805_2012Metric_Pad1.18x1.45mm_HandSolder, symbol Device:C
- added C3, C5: C, symbol Device:C
- added U5: AP2112K-3.3, Package_TO_SOT_SMD:SOT-23-5, symbol Regulator_Linear:AP2112K-3.3
Connections:
- net +5V: now also C3.1, U5.1 (VIN), U5.3 (EN)
- net 3.3V: now also C11.1, C5.1, U5.5 (VOUT)
- net GND: now also BT1.N2, U4.1 (GND), C11.2, C3.2, C5.2, U5.2 (GND)
- net at BT1.N1: now also BT1.P2
- no-connect marks 29 -> 25
Other:
- note added: "- OR -"
- moved on the sheet: C4, J4

Commit message: I swear this is the last PCB revision
Parts:
- added C999b1: C, Capacitor_SMD:C_0805_2012Metric_Pad1.18x1.45mm_HandSolder, symbol DisplayLibrary(sketch):CAP_CERAMIC0603_NO
- added C999d1: C, Capacitor_SMD:C_0603_1608Metric, symbol DisplayLibrary(sketch):C_Small
- added MOL3: CASE_SW, Connector_Molex:Molex_KK-254_AE-6410-02A_1x02_P2.54mm_Vertical, symbol DisplayLibrary(sketch):SW_Push
- 5Vin1: symbol Connector:Barrel_Jack -> DisplayLibrary(sketch):Barrel_Jack
- BOOT1, RST1: value (Generic) Lab Kit -> Lab Kit
- C12: renamed from C4; symbol Device:C -> DisplayLibrary(sketch):C
- C12B1: renamed from C3; symbol Device:C -> DisplayLibrary(sketch):C
- C13: renamed from C11; symbol Device:C -> DisplayLibrary(sketch):C
- C13B1: renamed from C5; symbol Device:C -> DisplayLibrary(sketch):C
- MOL1: renamed from UP1; value SW_Push -> CASE_SW
- MOL2: renamed from DOWN1; value SW_Push -> CASE_SW
- MOL4: renamed from J4; value Molex -> Vin; symbol Connector:Conn_01x02_Pin -> DisplayLibrary(sketch):Conn_01x02_Pin
- U4: symbol Regulator_Linear:AMS1117-3.3 -> DisplayLibrary(sketch):AMS1117-3.3
- U5: symbol Regulator_Linear:AP2112K-3.3 -> DisplayLibrary(sketch):AP2112K-3.3
- renumbered C8 to C1, C9 to C10, C10 to C11, C7 to C2, C17 to C3, C14 to C4, C2 to C5, C1 to C6, C6 to C7, C13 to C8, C16 to C9, PC2 to PC1, R26 to R10, R25 to R11, R28 to R8, R29 to R9
Connections:
- net 3.3V: no longer C13B1.1, U5.5 (VOUT)
- net ADDRA_3V: now also U1.23 (IO21), U2.4 (A3); no longer U1.19 (IO11), U2.3 (A2)
- net ADDRB_3V: now also U1.24 (IO47), U2.3 (A2); no longer U1.18 (IO10), U2.4 (A3)
- net ADDRC_3V: now also U1.21 (IO13), U2.6 (A5); no longer U1.17 (IO9), U2.5 (A4)
- net ADDRD_3V: now also U1.22 (IO14), U2.5 (A4); no longer U1.5 (IO5), U2.6 (A5)
- net B2_3V: now also U1.25 (IO48); no longer U1.20 (IO12)
- net CLK: now also U2.12 (B7); no longer U2.13 (B6)
- net CLK_3V: now also U1.19 (IO11), U2.8 (A7); no longer U1.12 (IO8), U2.7 (A6)
- net G1_3V: now also U1.35 (IO42), U3.5 (A4); no longer U1.32 (IO39), U3.8 (A7)
- net G2_3V: now also U1.32 (IO39), U3.8 (A7); no longer U1.35 (IO42), U3.5 (A4)
- net GND: now also MOL3.1
- net LAT: now also U2.13 (B6); no longer U2.12 (B7)
- net LAT_3V: now also U1.20 (IO12), U2.7 (A6); no longer U1.11 (IO18), U2.8 (A7)
- net M1_A: now also U2.16 (B3); no longer U2.17 (B2)
- net M1_B: now also U2.17 (B2); no longer U2.16 (B3)
- net M1_C: now also U2.14 (B5); no longer U2.15 (B4)
- net M1_D: now also U2.15 (B4); no longer U2.14 (B5)
- net M1_G1: now also U3.15 (B4); no longer U3.12 (B7)
- net M1_G2: now also U3.12 (B7); no longer U3.15 (B4)
- net M1_R1: now also U3.14 (B5); no longer U3.11 (B8)
- net M1_R2: now also U3.11 (B8); no longer U3.14 (B5)
- net OE_3V: now also U1.18 (IO10); no longer U1.10 (IO17)
- net R1_3V: now also U1.34 (IO41), U3.6 (A5); no longer U1.31 (IO38), U3.9 (A8)
- net R2_3V: now also U1.31 (IO38), U3.9 (A8); no longer U1.34 (IO41), U3.6 (A5)
- net D13 renamed D9
- net D9: now also U1.17 (IO9); no longer U1.21 (IO13)
- net DOWN renamed A1
- net UP renamed A0
- new net: C13B1.1, U5.5 (VOUT)
- new net A2: MOL3.2, U1.10 (IO17)
- no-connect marks 25 -> 30
Other:
- note added: "3.3V REGULATOR"
- note added: "5V IN"
- note added: "BATTERY"
- note added: "Caps for screen power??"
- note added: "IDC OUTPUT"
- note added: "POWER & D09 LEDS"
- note added: "TACT SWITCHES (molex to case)"
- note added: "bulk"
- note added: "dcpl"
- note added: "neopxl LED (boot status)"
- note added: "ref:"
- note added: "spare IDC for debug"
- note removed: "Caps for screen power"
- note removed: "IDC OUTPUT (HUB75)"
- note removed: "POWER & D13 LEDS"
- note removed: "TACT SWITCHES"
- note removed: "TO DO: (this is all board exluded!)"
- note removed: "neopxl LED (bootloader)"
- note removed: "spare for debug (if space on board)"
- note removed: "this needs to be done properly:"
- moved on the sheet: 5Vin1, BOOT1, BT1, C1, C10, C11, C12, C12B1, C13, C13B1, C2, C4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

Commit message: e
Parts:
- removed C12, C13: C, Capacitor_SMD:C_0805_2012Metric_Pad1.18x1.45mm_HandSolder, symbol DisplayLibrary(sketch):C
- added C12, C13: C, Capacitor_SMD:C_0805_2012Metric_Pad1.18x1.45mm_HandSolder, symbol DisplayLibrary(sketch):CAP_CERAMIC0603_NO
Connections:
- net +5V: now also C12.1
- net 3.3V: now also C13.1
- net GND: now also C12.2, C13.2
Changed lines of the file:
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@@
 	)
 	(junction
-		(at 86.36 129.54)
-		(diameter 0)
-		(color 0 0 0 0)
-	)
-	(junction
-		(at 107.95 129.54)
-		(diameter 0)
-		(color 0 0 0 0)
-	)
-	(junction
 		(at 86.36 161.29)
 		(diameter 0)
@@
 	)
 	(junction
+		(at 86.36 129.54)
+		(diameter 0)
+		(color 0 0 0 0)
+	)
+	(junction
 		(at 105.41 82.55)
 		(diameter 0)
 		(color 0 0 0 0)
 	)
+	(junction
+		(at 107.95 129.54)
+		(diameter 0)
+		(color 0 0 0 0)
+	)
 	(no_connect
 		(at 274.32 83.82)
@@
 	)
 	(symbol
+		(lib_id "DisplayLibrary(sketch):CAP_CERAMIC0603_NO")
+		(at 86.36 134.62 0)
+		(unit 1)
+		(exclude_from_sim no)
+		(in_bom yes)
+		(on_board yes)
+		(dnp no)
+		(property "Reference" "C12"
+			(at 89.916 133.35 0)
+			(effects
+				(font
+					(size 1.27 1.27)
+				)
+			)
+		)
+		(property "Value" "C"
+			(at 89.916 135.382 0)
+			(effects
+				(font
+					(size 1.27 1.27)
+				)
+			)
+		)
+		(property "Footprint" "Capacitor_SMD:C_0805_2012Metric_Pad1.18x1.45mm_HandSolder"
+			(at 86.36 134.62 0)
+			(effects
+				(font
+					(size 1.27 1.27)
+				)
+				(hide yes)
+			)
+		)
+		(property "Datasheet" ""
+			(at 86.36 134.62 0)
+			(effects
+				(font
+					(size 1.27 1.27)
+				)
+				(hide yes)
+			)
+		)
+		(property "Description" ""
+			(at 86.36 134.62 0)
+			(effects
+				(font
+					(size 1.27 1.27)
+				)
+				(hide yes)
+			)
+		)
+		(pin "1"
+		)
+		(pin "2"
+		)
+		(instances
+			(project "DisplayDriver"
+				(path "/ddc4c194-bb30-4734-adb1-ce29ad370a60"
+					(reference "C12")
+					(unit 1)
+				)
+			)
+		)
+	)
+	(symbol
 		(lib_id "DisplayLibrary(sketch):CAP_CERAMIC0805-NOOUTLINE")
 		(at 77.47 63.5 180)
@@
 	(symbol
 		(lib_id "DisplayLibrary(sketch):C")
-		(at 86.36 133.35 0)
-		(unit 1)
-		(exclude_from_sim no)
-		(in_bom yes)
-		(on_board yes)
-		(dnp no)
-		(property "Reference" "C12"
-			(at 88.646 133.35 0)
-			(effects
-				(font
-					(size 1.27 1.27)
-				)
-				(justify left)
-			)
-		)
-		(property "Value" "C"
-			(at 88.646 135.89 0)
-			(effects
-				(font
-					(size 1.27 1.27)
-				)
-				(justify left)
-			)
-		)
-		(property "Footprint" "Capacitor_SMD:C_0805_2012Metric_Pad1.18x1.45mm_HandSolder"
-			(at 87.3252 137.16 0)
-			(effects
-				(font
-					(size 1.27 1.27)
-				)
-				(hide yes)
-			)
-		)
-		(property "Datasheet" "~"
-			(at 86.36 133.35 0)
-			(effects
-				(font
-					(size 1.27 1.27)
-				)
-				(hide yes)
-			)
-		)
-		(property "Description" "Unpolarized capacitor"
-			(at 86.36 133.35 0)
-			(effects
-				(font
-					(size 1.27 1.27)
-				)
-				(hide yes)
-			)
-		)
-		(pin "2"
-		)
-		(pin "1"
-		)
-		(instances
-			(project "DisplayDriver"
-				(path "/ddc4c194-bb30-4734-adb1-ce29ad370a60"
-					(reference "C12")
-					(unit 1)
-				)
-			)
-		)
-	)
-	(symbol
-		(lib_id "DisplayLibrary(sketch):C")
 		(at 86.36 166.37 0)
 		(unit 1)
@@
 	)
 	(symbol
-		(lib_id "DisplayLibrary(sketch):C")
-		(at 107.95 133.35 0)
-		(unit 1)
-		(exclude_from_sim no)
-		(in_bom yes)
-		(on_board yes)
-		(dnp no)
-		(property "Reference" "C13"
-			(at 110.998 133.35 0)
-			(effects
-				(font
-					(size 1.27 1.27)
-				)
-				(justify left)
-			)
-		)
-		(property "Value" "C"
-			(at 110.998 135.89 0)
-			(effects
-				(font
-					(size 1.27 1.27)
-				)
-				(justify left)
-			)
-		)
-		(property "Footprint" "Capacitor_SMD:C_0805_2012Metric_Pad1.18x1.45mm_HandSolder"
-			(at 108.9152 137.16 0)
-			(effects
-				(font
-					(size 1.27 1.27)
-				)
-				(hide yes)
-			)
-		)
-		(property "Datasheet" "~"
-			(at 107.95 133.35 0)
-			(effects
-				(font
-					(size 1.27 1.27)
-				)
-				(hide yes)
-			)
-		)
-		(property "Description" "Unpolarized capacitor"
-			(at 107.95 133.35 0)
-			(effects
-				(font
-					(size 1.27 1.27)
-				)
-				(hide yes)
-			)
-		)
-		(pin "2"
-		)
-		(pin "1"
-		)
-		(instances
-			(project "DisplayDriver"
-				(path "/ddc4c194-bb30-4734-adb1-ce29ad370a60"
-					(reference "C13")
-					(unit 1)
-				)
-			)
-		)
-	)
-	(symbol
 		(lib_id "DisplayLibrary(sketch):PowerTags_+5V")
 		(at 77.47 31.75 0)
@@
 					(unit 1)
 				)
+			)
+		)
+	)
+	(symbol
+		(lib_id "DisplayLibrary(sketch):CAP_CERAMIC0603_NO")
+		(at 107.95 134.62 0)
+		(unit 1)
+		(exclude_from_sim no)
+		(in_bom yes)
+		(on_board yes)
+		(dnp no)
+		(property "Reference" "C13"
+			(at 111.506 133.35 0)
+			(effects
+				(font
+					(size 1.27 1.27)
+				)
+			)
+		)
+		(property "Value" "C"
+			(at 111.506 135.382 0)
+			(effects
+				(font
+					(size 1.27 1.27)
+				)
+			)
+		)
+		(property "Footprint" "Capacitor_SMD:C_0805_2012Metric_Pad1.18x1.45mm_HandSolder"
+			(at 107.95 134.62 0)
+			(effects
+				(font
+					(size 1.27 1.27)
+				)
+				(hide yes)
+			)
+		)
+		(property "Datasheet" ""
+			(at 107.95 134.62 0)
+			(effects
+				(font
+					(size 1.27 1.27)
+				)
+				(hide yes)
+			)
+		)
+		(property "Description" ""
+			(at 107.95 134.62 0)
+			(effects
+				(font
+					(size 1.27 1.27)
+				)
+				(hide yes)
+			)
+		)
+		(pin "1"
+		)
+		(pin "2"
+		)
+		(instances
+			(project "DisplayDriver"
+				(path "/ddc4c194-bb30-4734-adb1-ce29ad370a60"
+					(reference "C13")
+					(unit 1)
+				)

Commit message: bill of mat.
Parts:
- renumbered R11 to R10, R6 to R3, R7 to R6, R8 to R7, R9 to R8, R10 to R9
Changed lines of the file:
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@@
 		(on_board yes)
 		(dnp no)
-		(property "Reference" "R10"
+		(property "Reference" "R9"
 			(at 50.292 154.686 90)
 			(effects
@@
 			(project "DisplayDriver"
 				(path "/ddc4c194-bb30-4734-adb1-ce29ad370a60"
-					(reference "R10")
+					(reference "R9")
 					(unit 1)
 				)
@@
 		(on_board yes)
 		(dnp no)
-		(property "Reference" "R9"
+		(property "Reference" "R8"
 			(at 53.086 141.732 90)
 			(effects
@@
 			(project "DisplayDriver"
 				(path "/ddc4c194-bb30-4734-adb1-ce29ad370a60"
-					(reference "R9")
+					(reference "R8")
 					(unit 1)
 				)
@@
 			)
 		)
-		(property "Datasheet" ""
+		(property "Datasheet" "~"
 			(at 167.64 74.93 0)
 			(effects
@@
 		(on_board yes)
 		(dnp no)
-		(property "Reference" "R7"
+		(property "Reference" "R6"
 			(at 181.864 59.436 0)
 			(effects
@@
 			(project ""
 				(path "/ddc4c194-bb30-4734-adb1-ce29ad370a60"
-					(reference "R7")
+					(reference "R6")
 					(unit 1)
 				)
@@
 		(on_board yes)
 		(dnp no)
-		(property "Reference" "R6"
+		(property "Reference" "R3"
 			(at 150.114 72.898 90)
 			(effects
@@
 			)
 		)
-		(property "Datasheet" ""
+		(property "Datasheet" "~"
 			(at 147.32 74.93 0)
 			(effects
@@
 			(project "DisplayDriver"
 				(path "/ddc4c194-bb30-4734-adb1-ce29ad370a60"
-					(reference "R6")
+					(reference "R3")
 					(unit 1)
 				)
@@
 			)
 		)
-		(property "Datasheet" ""
+		(property "Datasheet" "~"
 			(at 157.48 62.23 0)
 			(effects
@@
 			)
 		)
-		(property "Datasheet" ""
+		(property "Datasheet" "~"
 			(at 201.93 22.86 0)
 			(effects
@@
 		(on_board yes)
 		(dnp no)
-		(property "Reference" "R8"
+		(property "Reference" "R7"
 			(at 53.086 134.874 90)
 			(effects
@@
 			(project "DisplayDriver"
 				(path "/ddc4c194-bb30-4734-adb1-ce29ad370a60"
-					(reference "R8")
+					(reference "R7")
 					(unit 1)
 				)
@@
 			)
 		)
-		(property "Datasheet" ""
+		(property "Datasheet" "~"
 			(at 194.31 62.23 0)
 			(effects
@@
 			)
 		)
-		(property "Datasheet" ""
+		(property "Datasheet" "~"
 			(at 153.67 24.13 0)
 			(effects
@@
 		(on_board yes)
 		(dnp no)
-		(property "Reference" "R11"
+		(property "Reference" "R10"
 			(at 53.848 162.306 90)
 			(effects
@@
 			(project "DisplayDriver"
 				(path "/ddc4c194-bb30-4734-adb1-ce29ad370a60"
-					(reference "R11")
+					(reference "R10")
 					(unit 1)
 				)

Commit message: pcb review prep
Other:
- note added: "bulk 75HCT"
- note added: "bulk ESP (2x)"
- note added: "bulk Neopix"
- note added: "dcpl ESP"
- note added: "dcpl Neopix"
- note removed: "bulk"
- note removed: "bulk ESP"
- note removed: "dcpl"
- moved on the sheet: C4, C5, C6, C8, C9

Commit message: DD3 (+josh stuff)
Parts:
- removed C12B1, C13B1: C, symbol DisplayLibrary(sketch):C
- removed U5: AP2112K-3.3, Package_TO_SOT_SMD:SOT-23-5, symbol DisplayLibrary(sketch):AP2112K-3.3
Connections:
- no-connect marks 30 -> 29
Other:
- note removed: "- OR -"
- company: Aviator -> Aviator - DT
- title: Display Driver -> Display Driver (Main PCB)
- moved on the sheet: C1, C10, C11, C2, C3, C4, C5, C6, C8, C9, PC1, U2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
